File: mcu.kicad_sch (KiCad schematic)
At the start: 75 parts, among them J12 292161-3, J7 Conn_02x10_Odd_Even, J8 TagConnect_TC2050, J9 292161-3, SW1 SW_Push, SW2 SW_Push, U10 PCA9548APW, U11 AZ1117H-1.8TRE1_SOT223, U50 TMP102xxDRL, U51 TMP102xxDRL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

Commit message: MCU I2C4 is now directly connected to clock control
Connections:
- net CLK_CTL_I2C_SCL: now also U7.54 (PF14); no longer U10.18 (SC6)
- net CLK_CTL_I2C_SDA: now also U7.55 (PF15); no longer U10.17 (SD6)
- no-connect marks 75 -> 73
Other:
- note added: "I2C4 is dedicated to clock"
- note added: "Variable voltage for SYZYGY"
- note added: "slave I2C from SOC/Linux +3V3 / PS500"
- note removed: "master I2C to control the SOC/Linux +3V3 / PS500"
- moved on the sheet: R86
