File: mcu.kicad_sch (KiCad schematic)
At the start: 75 parts, among them J12 292161-3, J7 Conn_02x10_Odd_Even, J8 TagConnect_TC2050, J9 292161-3, SW1 SW_Push, SW2 SW_Push, U10 PCA9548APW, U11 AZ1117H-1.8TRE1_SOT223, U50 TMP102xxDRL, U51 TMP102xxDRL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

Commit message: schema: U8 I2C EEPROM line correction
Connections:
- net I2C_MCU_EEP_SCL: now also U10.20 (SC7); no longer U10.19 (SD7)
- net I2C_MCU_EEP_SDA: now also U10.19 (SD7); no longer U10.20 (SC7)

Commit message: schema: JTAG connector & resistors, rev change
Parts:
- added R393, R394: 150, Resistor_SMD:R_0402_1005Metric, symbol Device:R_Small
Connections:
- net NJTRST: now also R393.2
- net NRST: now also R394.2
- new net: J8.9 (nTRST), R393.1, R394.1
Other:
- moved on the sheet: R100, R103, R104, R99
Changed lines of the file:
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@@
 		(title "NASR-M")
 		(date "2025-10-22")
-		(rev "D 0.9.5")
+		(rev "D 0.9.8")
 		(company "electrodyssey.net")
 		(comment 1 "Board MCU controlls the VIO power and SYZYGY ports")
@@
 		(comment 3 "Author: Nazim Aghabayov")
 		(comment 4 "SYZYGY Carrier Mainboard")
-		(comment 5 "rel: Fletched Bustard")
+		(comment 5 "rel: Wild Goose")
 	)
