File: mcu.kicad_sch (KiCad schematic)
At the start: 77 parts, among them J12 292161-3, J7 Conn_02x10_Odd_Even, J8 TagConnect_TC2050, J9 292161-3, SW1 SW_Push, SW2 SW_Push, U10 PCA9548APW, U11 AZ1117H-1.8TRE1_SOT223, U50 TMP102xxDRL, U51 TMP102xxDRL, U7 STM32H723ZGTx, U8 24AA02E48T-I/OT, U9 TXS0108EPW, Y1 8MHz, Y2 32.768KHz

Commit message: MCU TagConnect nRST, SATA socket
MCU TagConnect now connects to NRST net of the MCU.
SATA socket is not DNP any more
Parts:
- R393: now not fitted
- R394: now fitted
