File: psu.kicad_sch (KiCad schematic)
At the start: 76 parts, among them J1 39-28-1243, J2 292161-3, J3 292161-3, J4 292161-3, J5 292161-3, J6 292161-3, Q1 IRLML6344TRPBF, Q2 BSS138, Q3 IRLML6344TRPBF, Q4 IRLML6344TRPBF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

Commit message: JLCPCB part id's update
Parts:
- FAN50x50-12V1:  LCSC Part # (none) -> C456906
- J1: JLCPCB Part # (none) -> C22365710; Manufacturer_Part_Number 39-28-1243 -> DLL-5566-24A
- R22: JLCPCB Part # C3152375 -> C5154013; Part SC1210J3300F1CNRH -> FRC1210J331TS
Changed lines of the file:
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@@
 			)
 		)
-		(property "JLCPCB Part #" "C3152375"
+		(property "JLCPCB Part #" "C5154013"
 			(at 337.82 219.71 0)
 			(effects
@@
 			)
 		)
-		(property "Part" "SC1210J3300F1CNRH"
+		(property "Part" "FRC1210J331TS"
 			(at 337.82 219.71 90)
 			(effects
@@
 			)
 		)
-		(property "Description" "50X50X10 SUNON MF50101V2-1000U-A99 maglev fan"
+		(property "Description" "50X50X10 SUNON MF50101V2-1000U-A99 maglev fan; alt: MF50100V1-1000C-A99"
 			(at 324.612 82.55 0)
 			(effects
@@
 			)
 		)
+		(property " LCSC Part #" "C456906"
+			(at 313.69 88.9 0)
+			(effects
+				(font
+					(size 1.27 1.27)
+				)
+				(hide yes)
+			)
+		)
 		(instances
 			(project "NASR"
@@
 			)
 		)
-		(property "Manufacturer_Part_Number" "39-28-1243"
+		(property "Manufacturer_Part_Number" "DLL-5566-24A"
 			(at 57.15 818.415 0)
 			(effects
@@
 			)
 		)
-		(property "JLCPCB Part #" ""
+		(property "JLCPCB Part #" "C22365710"
 			(at 38.1 23.495 0)
 			(effects
