File: psu.kicad_sch (KiCad schematic)
At the start: 76 parts, among them J1 39-28-1243, J2 292161-3, J3 292161-3, J4 292161-3, J5 292161-3, J6 292161-3, Q1 IRLML6344TRPBF, Q2 BSS138, Q3 IRLML6344TRPBF, Q4 IRLML6344TRPBF, U1 AZ1117-3.3

Commit message: bom: substitute out-of-stock passives, sync descriptions to JLCPCB IDs
Every substitution keeps its existing footprint, so no PCB rework is
implied. Stock figures verified against live LCSC, not the parts-library
snapshot (which was stale on four parts).

  C11-C13  C188358 -> C178366   82uF/35V -> 180uF/25V OS-CON SVPF (was OOS)
  R54      C138285 -> C2933137  12.7k 0603 (was OOS)
  31x tant C1954274 -> C7214    22uF 16V -> 25V; ~16 -> ~2580 boards of
                                stock, and fixes the +12VEXT derating on
                                C430/C431 (75% -> 48% of rating)
  20x cap  C513774 -> C13585    10uF 1206, JLC Basic part
  C76,C77  C2918589 -> C541338  4.3pF +-0.1pF, 32.768kHz load caps for Y2
  R286     C705904 -> C2930124  649R, HX2VL RREF
  R45      C2936632 -> C17477   consolidated onto an existing BOM line
  C328     C2170363 -> C368809  consolidated; was outside the JLC library
  R172     C705658 -> C705678   consolidated; was outside the JLC library

Fix eight capacitors labelled 10nFx50V that carried a 10uF part number:
C31 C32 C302 C307 C309 C347 C360 C368 -> value corrected to 10uFx50V.
All sit on power rails or LDO inputs where 10uF is the intent.

Restore C302's Footprint, which had been corrupted to "c9" (not a valid
library reference; would have failed the next PCB update).

Regenerate Description on all 822 R/C from live LCSC parametric data so
each matches its JLCPCB Part #.

Value fields keep the project convention: the voltage suffix is the design
minimum, not the fitted part's rating, so the tantalum stayed 22uFx16V.
C11-C13 did change 82uF -> 180uF because the capacitance itself changed.

Also carries work in progress from this session: H35 mounting hole,
R50/R137/R285 moved to 0402 (C25792), R30 220R -> 330R (C5154013),
C24 -> C1618.

NASR.net and NASR.kicad_pcb still predate these schematic edits; they need
a netlist re-export and Update PCB from Schematic.

Co-Authored-By: Claude Opus 5 (1M context) <noreply@anthropic.c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
Parts:
- C11, C12, C13: value 82uF -> 180uF; JLCPCB Part # C188358 -> C178366; Part 35SVPF82M -> 25SVPF180M
- C14, C8: JLCPCB Part # C513774 -> C13585; Part CS3216X5R106K500NRI -> CL31A106KBHNNNE
- R30: value 220 -> 330; JLCPCB Part # C230115 -> C5154013; Part AC1210FR-07220RL -> FRC1210J331TS
Changed lines of the file:
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@@
 			)
 		)
-		(property "Description" ""
+		(property "Description" "50V 100nF X7R ±10% 0805 Multilayer Ceramic Capacitors MLCC - SMD/SMT ROHS"
 			(at 111.76 124.46 0)
 			(effects
@@
 			)
 		)
-		(property "Description" ""
+		(property "Description" "-55℃~+155℃ 10kΩ 50V 62.5mW Thick Film Resistor ±1% ±100ppm/℃ 0402 Chip Resistor - Surface Mount ROHS"
 			(at 365.76 143.51 0)
 			(effects
@@
 			)
 		)
-		(property "Description" ""
+		(property "Description" "50V 100nF X7R ±10% 0805 Multilayer Ceramic Capacitors MLCC - SMD/SMT ROHS"
 			(at 35.56 170.18 0)
 			(effects
@@
 			)
 		)
-		(property "Value" "82uF"
+		(property "Value" "180uF"
 			(at 100.838 170.9039 0)
 			(effects
@@
 			)
 		)
-		(property "Description" ""
+		(property "Description" "25V 180uF ±20% SMD,D8xL11.9mm Aluminum Electrolytic Capacitors - SMD ROHS"
 			(at 97.79 170.18 0)
 			(effects
@@
 			)
 		)
-		(property "Part" "35SVPF82M "
+		(property "Part" "25SVPF180M"
 			(at 97.79 170.18 0)
 			(effects
@@
 			)
 		)
-		(property "JLCPCB Part #" "C188358"
+		(property "JLCPCB Part #" "C178366"
 			(at 97.79 170.18 0)
 			(effects
@@
 			)
 		)
-		(property "Description" "-55℃~+155℃ 200V 250mW 330Ω Thick Film Resistor ±1% ±100ppm/℃ 1206 Chip Resistor - Surface Mount ROHS"
+		(property "Description" "-55℃~+155℃ 330Ω 200V 250mW Thick Film Resistor ±1% ±100ppm/℃ 1206 Chip Resistor - Surface Mount ROHS"
 			(at 133.35 78.74 0)
 			(effects
@@
 			)
 		)
-		(property "Description" ""
+		(property "Description" "-55℃~+155℃ 10kΩ 50V 62.5mW Thick Film Resistor ±1% ±100ppm/℃ 0402 Chip Resistor - Surface Mount ROHS"
 			(at 365.76 81.28 0)
 			(effects
@@
 			)
 		)
-		(property "Description" "-55℃~+155℃ 100mW 10kΩ 75V Thick Film Resistor ±1% ±100ppm/℃ 0603 Chip Resistor - Surface Mount ROHS"
+		(property "Description" "-55℃~+155℃ 10kΩ 75V 100mW Thick Film Resistor ±1% ±100ppm/℃ 0603 Chip Resistor - Surface Mount ROHS"
 			(at 196.85 73.66 0)
 			(effects
@@
 			)
 		)
-		(property "Description" ""
+		(property "Description" "50V 10uF X5R ±10% 1206 Multilayer Ceramic Capacitors MLCC - SMD/SMT ROHS"
 			(at 50.8 265.43 0)
 			(effects
@@
 			)
 		)
-		(property "Part" "CS3216X5R106K500NRI"
+		(property "Part" "CL31A106KBHNNNE"
 			(at 50.8 265.43 0)
 			(effects
@@
 			)
 		)
-		(property "JLCPCB Part #" "C513774"
+		(property "JLCPCB Part #" "C13585"
 			(at 50.8 265.43 0)
 			(effects
@@
 			)
 		)
-		(property "Description" "10nF 1kV X7R ±10% 1206 Multilayer Ceramic Capacitors MLCC - SMD/SMT ROHS"
+		(property "Description" "1kV 10nF X7R ±10% 1206 Multilayer Ceramic Capacitors MLCC - SMD/SMT ROHS"
 			(at 58.42 271.78 0)
 			(effects
@@
 			)
 		)
-		(property "Description" ""
+		(property "Description" "25V 100nF X7R ±5% 0402 Multilayer Ceramic Capacitors MLCC - SMD/SMT ROHS"
 			(at 80.01 90.17 0)
 			(effects
@@
 			)
 		)
-		(property "Description" ""
+		(property "Description" "330Ω 200V 500mW Thick Film Resistor ±5% ±100ppm/℃ 1210 Chip Resistor - Surface Mount ROHS"
 			(at 337.82 219.71 0)
 			(effects
@@
 			)
 		)
-		(property "Description" ""
+		(property "Description" "-55℃~+155℃ 330Ω 75V 100mW Thick Film Resistor ±1% ±100ppm/℃ 0603 Chip Resistor - Surface Mount ROHS"
 			(at 214.63 119.38 0)
 			(effects
@@
 			)
 		)
-		(property "Description" ""
+		(property "Description" "-55℃~+155℃ 330Ω 75V 100mW Thick Film Resistor ±1% ±100ppm/℃ 0603 Chip Resistor - Surface Mount ROHS"
 			(at 246.38 120.65 0)
 			(effects
@@
 			)
 		)
-		(property "Description" ""
+		(property "Description" "50V 100nF X7R ±10% 0805 Multilayer Ceramic Capacitors MLCC - SMD/SMT ROHS"
 			(at 111.76 215.9 0)
 			(effects
@@
 			)
 		)
-		(property "Description" ""
+		(property "Description" "-55℃~+155℃ 150Ω 50V 62.5mW Thick Film Resistor ±1% ±100ppm/℃ 0402 Chip Resistor - Surface Mount ROHS"
 			(at 355.6 76.2 0)
 			(effects
@@
 			)
 		)
-		(property "Description" ""
+		(property "Description" "50V 100nF X7R ±10% 0805 Multilayer Ceramic Capacitors MLCC - SMD/SMT ROHS"
 			(at 111.76 170.18 0)
 			(effects
@@
 			)
 		)
-		(property "Description" ""
+		(property "Description" "-55℃~+155℃ 150Ω 50V 62.5mW Thick Film Resistor ±1% ±100ppm/℃ 0402 Chip Resistor - Surface Mount ROHS"
 			(at 88.9 83.82 0)
 			(effects
@@
 			)
 		)
-		(property "Description" ""
+		(property "Description" "-55℃~+155℃ 1kΩ 50V 62.5mW Thick Film Resistor ±1% ±100ppm/℃ 0402 Chip Resistor - Surface Mount ROHS"
 			(at 24.13 77.47 0)
 			(effects
@@
 			)
 		)
-		(property "Description" ""
+		(property "Description" "50V 100nF X7R ±10% 0805 Multilayer Ceramic Capacitors MLCC - SMD/SMT ROHS"
 			(at 114.3 266.7 0)
 			(effects
@@
 			)
 		)
-		(property "Description" ""
+		(property "Description" "-55℃~+155℃ 1kΩ 50V 62.5mW Thick Film Resistor ±1% ±100ppm/℃ 0402 Chip Resistor - Surface Mount ROHS"
 			(at 69.85 91.44 0)
 			(effects
@@
 			)
 		)
-		(property "Description" ""
+		(property "Description" "-55℃~+155℃ 1kΩ 50V 62.5mW Thick Film Resistor ±1% ±100ppm/℃ 0402 Chip Resistor - Surface Mount ROHS"
 			(at 232.41 119.38 0)
 			(effects
@@
 			)
 		)
-		(property "Description" ""
+		(property "Description" "-55℃~+155℃ 150Ω 50V 62.5mW Thick Film Resistor ±1% ±100ppm/℃ 0402 Chip Resistor - Surface Mount ROHS"
 			(at 359.41 138.43 0)
 			(effects
@@
 			)
 		)
-		(property "Value" "220"
+		(property "Value" "330"
 			(at 365.506 220.98 0)
 			(effects
@@
 			)
 		)
-		(property "Description" ""
+		(property "Description" "330Ω 200V 500mW Thick Film Resistor ±5% ±100ppm/℃ 1210 Chip Resistor - Surface Mount ROHS"
 			(at 372.11 219.71 0)
 			(effects
@@
 			)
 		)
-		(property "JLCPCB Part #" "C230115"
+		(property "JLCPCB Part #" "C5154013"
 			(at 372.11 219.71 0)
 			(effects
@@
 			)
 		)
-		(property "Part" "AC1210FR-07220RL"
+		(property "Part" "FRC1210J331TS"
 			(at 372.11 219.71 90)
 			(effects
@@
 			)
 		)
-		(property "Description" ""
+		(property "Description" "50V 10uF X5R ±10% 1206 Multilayer Ceramic Capacitors MLCC - SMD/SMT ROHS"
 			(at 105.41 266.7 0)
 			(effects
@@
 			)
 		)
-		(property "Part" "CS3216X5R106K500NRI"
+		(property "Part" "CL31A106KBHNNNE"
 			(at 105.41 266.7 0)
 			(effects
@@
 			)
 		)
-		(property "JLCPCB Part #" "C513774"
+		(property "JLCPCB Part #" "C13585"
 			(at 105.41 266.7 0)
 			(effects
@@
 			)
 		)
-		(property "Description" ""
+		(property "Description" "-55℃~+155℃ 4.7kΩ 50V 62.5mW Thick Film Resistor ±1% ±100ppm/℃ 0402 Chip Resistor - Surface Mount ROHS"
 			(at 345.44 132.08 0)
 			(effects
@@
 			)
 		)
-		(property "Description" ""
+		(property "Description" "35V 1uF X7R ±10% 0603 Multilayer Ceramic Capacitors MLCC - SMD/SMT ROHS"
 			(at 22.86 92.71 0)
 			(effects
@@
 			)
 		)
-		(property "Description" ""
+		(property "Description" "50V 100nF X7R ±10% 0805 Multilayer Ceramic Capacitors MLCC - SMD/SMT ROHS"
 			(at 35.56 215.9 0)
 			(effects
@@
 			)
 		)
-		(property "Description" ""
+		(property "Description" "-55℃~+155℃ 1kΩ 50V 62.5mW Thick Film Resistor ±1% ±100ppm/℃ 0402 Chip Resistor - Surface Mount ROHS"
 			(at 40.64 90.17 0)
 			(effects
@@
 			)
 		)
-		(property "Value" "82uF"
+		(property "Value" "180uF"
 			(at 100.838 125.1839 0)
 			(effects
@@
 			)
 		)
-		(property "Description" ""
+		(property "Description" "25V 180uF ±20% SMD,D8xL11.9mm Aluminum Electrolytic Capacitors - SMD ROHS"
 			(at 97.79 124.46 0)
 			(effects
@@
 			)
 		)
-		(property "Part" "35SVPF82M "
+		(property "Part" "25SVPF180M"
 			(at 97.79 124.46 0)
 			(effects
@@
 			)
 		)
-		(property "JLCPCB Part #" "C188358"
+		(property "JLCPCB Part #" "C178366"
 			(at 97.79 124.46 0)
 			(effects
@@
 			)
 		)
-		(property "Description" "-55℃~+155℃ 200V 250mW 330Ω Thick Film Resistor ±1% ±100ppm/℃ 1206 Chip Resistor - Surface Mount ROHS"
+		(property "Description" "-55℃~+155℃ 330Ω 200V 250mW Thick Film Resistor ±1% ±100ppm/℃ 1206 Chip Resistor - Surface Mount ROHS"
 			(at 104.14 74.93 0)
 			(effects
@@
 			)
 		)
-		(property "Description" "-55℃~+155℃ 100mW 10kΩ 75V Thick Film Resistor ±1% ±100ppm/℃ 0603 Chip Resistor - Surface Mount ROHS"
+		(property "Description" "-55℃~+155℃ 10kΩ 75V 100mW Thick Film Resistor ±1% ±100ppm/℃ 0603 Chip Resistor - Surface Mount ROHS"
 			(at 218.44 73.66 0)
 			(effects
@@
 			)
 		)
-		(property "Description" ""
+		(property "Description" "-55℃~+155℃ 10kΩ 50V 62.5mW Thick Film Resistor ±1% ±100ppm/℃ 0402 Chip Resistor - Surface Mount ROHS"
 			(at 80.01 77.47 0)
 			(effects
@@
 			)
 		)
-		(property "Description" ""
+		(property "Description" "-55℃~+155℃ 4.7kΩ 50V 62.5mW Thick Film Resistor ±1% ±100ppm/℃ 0402 Chip Resistor - Surface Mount ROHS"
 			(at 345.44 71.12 0)
 			(effects
@@
 			)
 		)
-		(property "Value" "82uF"
+		(property "Value" "180uF"
 			(at 100.838 216.6239 0)
 			(effects
@@
 			)
 		)
-		(property "Description" ""
+		(property "Description" "25V 180uF ±20% SMD,D8xL11.9mm Aluminum Electrolytic Capacitors - SMD ROHS"
 			(at 97.79 215.9 0)
 			(effects
@@
 			)
 		)
-		(property "Part" "35SVPF82M "
+		(property "Part" "25SVPF180M"
 			(at 97.79 215.9 0)
 			(effects
@@
 			)
 		)
-		(property "JLCPCB Part #" "C188358"
+		(property "JLCPCB Part #" "C178366"
 			(at 97.79 215.9 0)
 			(effects
@@
 			)
 		)
-		(property "Description" ""
+		(property "Description" "50V 100nF X7R ±10% 0805 Multilayer Ceramic Capacitors MLCC - SMD/SMT ROHS"
 			(at 35.56 124.46 0)
 			(effects
@@
 			)
 		)
-		(property "Description" ""
+		(property "Description" "50V 100nF X7R ±10% 0805 Multilayer Ceramic Capacitors MLCC - SMD/SMT ROHS"
 			(at 30.48 264.16 0)
 			(effects
@@
 			)
 		)
-		(property "Description" ""
+		(property "Description" "-55℃~+155℃ 10kΩ 50V 62.5mW Thick Film Resistor ±1% ±100ppm/℃ 0402 Chip Resistor - Surface Mount ROHS"
 			(at 95.25 88.9 0)
 			(effects
