File: psu.kicad_sch (KiCad schematic)
At the start: 76 parts, among them J1 39-28-1243, J2 292161-3, J3 292161-3, J4 292161-3, J5 292161-3, J6 292161-3, Q1 IRLML6344TRPBF, Q2 BSS138, Q3 IRLML6344TRPBF, Q4 IRLML6344TRPBF, U1 AZ1117-3.3

Commit message: JLCPCB ID attribute updates
These 'JLCPCB Part #' updates reflect the JLCPCB assembly order # SMT026073061946-2250854A
Parts:
- R23, R24: JLCPCB Part # C25900 -> C105871; Part 0402WGF4701TCE -> RC0402FR-074K7L
Changed lines of the file:
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@@
 			)
 		)
-		(property "JLCPCB Part #" "C25900"
+		(property "JLCPCB Part #" "C105871"
 			(at 345.44 132.08 0)
 			(effects
@@
 			)
 		)
-		(property "Part" "0402WGF4701TCE"
+		(property "Part" "RC0402FR-074K7L"
 			(at 345.44 132.08 0)
 			(effects
@@
 			)
 		)
-		(property "JLCPCB Part #" "C25900"
+		(property "JLCPCB Part #" "C105871"
 			(at 345.44 71.12 0)
 			(effects
@@
 			)
 		)
-		(property "Part" "0402WGF4701TCE"
+		(property "Part" "RC0402FR-074K7L"
 			(at 345.44 71.12 0)
 			(effects
