File: sdio.kicad_sch (KiCad schematic)
At the start: 45 parts, among them IC4 TXS02612RTWR, J23 SCHA1B0100, U30 KLM8G1GETF-B041, U31 AZ1117H-1.8TRE1_SOT223

Commit message: JLCPCB part id's update
Parts:
- R251, R253: JLCPCB Part # C21189 -> C2906974; Part 0603WAF0000T5E -> FRC0603F0000TS
Changed lines of the file:
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@@
 			)
 		)
-		(property "JLCPCB Part #" "C21189"
+		(property "JLCPCB Part #" "C2906974"
 			(at 330.2 64.77 0)
 			(effects
@@
 			)
 		)
-		(property "Part" "0603WAF0000T5E"
+		(property "Part" "FRC0603F0000TS"
 			(at 330.2 64.77 90)
 			(effects
@@
 			)
 		)
-		(property "JLCPCB Part #" "C21189"
+		(property "JLCPCB Part #" "C2906974"
 			(at 351.79 176.53 0)
 			(effects
@@
 			)
 		)
-		(property "Part" "0603WAF0000T5E"
+		(property "Part" "FRC0603F0000TS"
 			(at 351.79 176.53 90)
 			(effects
