File: sdio.kicad_sch (KiCad schematic)
At the start: 45 parts, among them IC4 TXS02612RTWR, J23 SCHA1B0100, U30 KLM8G1GETF-B041, U31 AZ1117H-1.8TRE1_SOT223

Commit message: bom: substitute out-of-stock passives, sync descriptions to JLCPCB IDs
Every substitution keeps its existing footprint, so no PCB rework is
implied. Stock figures verified against live LCSC, not the parts-library
snapshot (which was stale on four parts).

  C11-C13  C188358 -> C178366   82uF/35V -> 180uF/25V OS-CON SVPF (was OOS)
  R54      C138285 -> C2933137  12.7k 0603 (was OOS)
  31x tant C1954274 -> C7214    22uF 16V -> 25V; ~16 -> ~2580 boards of
                                stock, and fixes the +12VEXT derating on
                                C430/C431 (75% -> 48% of rating)
  20x cap  C513774 -> C13585    10uF 1206, JLC Basic part
  C76,C77  C2918589 -> C541338  4.3pF +-0.1pF, 32.768kHz load caps for Y2
  R286     C705904 -> C2930124  649R, HX2VL RREF
  R45      C2936632 -> C17477   consolidated onto an existing BOM line
  C328     C2170363 -> C368809  consolidated; was outside the JLC library
  R172     C705658 -> C705678   consolidated; was outside the JLC library

Fix eight capacitors labelled 10nFx50V that carried a 10uF part number:
C31 C32 C302 C307 C309 C347 C360 C368 -> value corrected to 10uFx50V.
All sit on power rails or LDO inputs where 10uF is the intent.

Restore C302's Footprint, which had been corrupted to "c9" (not a valid
library reference; would have failed the next PCB update).

Regenerate Description on all 822 R/C from live LCSC parametric data so
each matches its JLCPCB Part #.

Value fields keep the project convention: the voltage suffix is the design
minimum, not the fitted part's rating, so the tantalum stayed 22uFx16V.
C11-C13 did change 82uF -> 180uF because the capacitance itself changed.

Also carries work in progress from this session: H35 mounting hole,
R50/R137/R285 moved to 0402 (C25792), R30 220R -> 330R (C5154013),
C24 -> C1618.

NASR.net and NASR.kicad_pcb still predate these schematic edits; they need
a netlist re-export and Update PCB from Schematic.

Co-Authored-By: Claude Opus 5 (1M context) <noreply@anthropic.c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
Parts:
- C293, C296, C299, C303, C305: JLCPCB Part # C513774 -> C13585; Part CS3216X5R106K500NRI -> CL31A106KBHNNNE
- C301, C308: JLCPCB Part # C1954274 -> C7214; Part TR3C226K016C0350 -> TAJC226K025RNJ
- C302, C307, C309: value 10nFx50V -> 10uFx50V; JLCPCB Part # C513774 -> C13585; Part (none) -> CL31A106KBHNNNE
Changed lines of the file:
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@@
 			)
 		)
-		(property "Description" ""
+		(property "Description" "50V 10uF X5R ±10% 1206 Multilayer Ceramic Capacitors MLCC - SMD/SMT ROHS"
 			(at 154.94 24.13 0)
 			(effects
@@
 			)
 		)
-		(property "Part" "CS3216X5R106K500NRI"
+		(property "Part" "CL31A106KBHNNNE"
 			(at 154.94 24.13 0)
 			(effects
@@
 			)
 		)
-		(property "JLCPCB Part #" "C513774"
+		(property "JLCPCB Part #" "C13585"
 			(at 154.94 24.13 0)
 			(effects
@@
 			)
 		)
-		(property "Description" ""
+		(property "Description" "25V 100nF X7R ±5% 0402 Multilayer Ceramic Capacitors MLCC - SMD/SMT ROHS"
 			(at 149.86 172.72 0)
 			(effects
@@
 			)
 		)
-		(property "Description" ""
+		(property "Description" "25V 100nF X7R ±5% 0402 Multilayer Ceramic Capacitors MLCC - SMD/SMT ROHS"
 			(at 351.79 196.85 0)
 			(effects
@@
 			)
 		)
-		(property "Description" ""
+		(property "Description" "25V 100nF X7R ±5% 0402 Multilayer Ceramic Capacitors MLCC - SMD/SMT ROHS"
 			(at 347.98 152.4 0)
 			(effects
@@
 			)
 		)
-		(property "Description" "-55℃~+125℃ 16V 22uF 350mΩ ±10% 2312 Tantalum Capacitors ROHS"
+		(property "Description" "25V 22uF ±10% CASE-C-6032-28(mm) Tantalum Capacitors ROHS"
 			(at 326.39 152.4 0)
 			(effects
@@
 			)
 		)
-		(property "Part" "TR3C226K016C0350"
+		(property "Part" "TAJC226K025RNJ"
 			(at 326.39 152.4 0)
 			(effects
@@
 			)
 		)
-		(property "JLCPCB Part #" "C1954274"
+		(property "JLCPCB Part #" "C7214"
 			(at 326.39 152.4 0)
 			(effects
@@
 			)
 		)
-		(property "Value" "10nFx50V"
+		(property "Value" "10uFx50V"
 			(at 336.55 153.6763 0)
 			(effects
@@
 			)
 		)
-		(property "Description" ""
+		(property "Description" "50V 10uF X5R ±10% 1206 Multilayer Ceramic Capacitors MLCC - SMD/SMT ROHS"
+			(at 334.01 152.4 0)
+			(effects
+				(font
+					(size 1.27 1.27)
+				)
+				(hide yes)
+			)
+		)
+		(property "JLCPCB Part #" "C13585"
 			(at 334.01 152.4 0)
 			(effects
@@
 			)
 		)
-		(property "JLCPCB Part #" "C513774"
+		(property "Part" "CL31A106KBHNNNE"
 			(at 334.01 152.4 0)
 			(effects
@@
 			)
 		)
-		(property "Description" ""
+		(property "Description" "25V 100nF X7R ±5% 0402 Multilayer Ceramic Capacitors MLCC - SMD/SMT ROHS"
 			(at 340.36 196.85 0)
 			(effects
@@
 			)
 		)
-		(property "Description" ""
+		(property "Description" "-55℃~+155℃ 150Ω 50V 62.5mW Thick Film Resistor ±1% ±100ppm/℃ 0402 Chip Resistor - Surface Mount ROHS"
 			(at 58.42 80.01 0)
 			(effects
@@
 			)
 		)
-		(property "Description" ""
+		(property "Description" "25V 100nF X7R ±5% 0402 Multilayer Ceramic Capacitors MLCC - SMD/SMT ROHS"
 			(at 64.77 36.83 0)
 			(effects
@@
 			)
 		)
-		(property "Description" ""
+		(property "Description" "-55℃~+155℃ 22.1Ω 50V 62.5mW Thick Film Resistor ±1% ±100ppm/℃ 0402 Chip Resistor - Surface Mount ROHS"
 			(at 59.69 64.77 0)
 			(effects
@@
 		(fields_autoplaced yes)
 		(property "Reference" "C302"
-			(at 264.16 228.6063 0)
+			(at 264.16 228.6062 0)
 			(effects
 				(font
@@
 			)
 		)
-		(property "Value" "10nFx50V"
-			(at 264.16 231.1463 0)
+		(property "Value" "10uFx50V"
+			(at 264.16 231.1462 0)
 			(effects
 				(font
@@
 			)
 		)
-		(property "Description" ""
+		(property "Description" "50V 10uF X5R ±10% 1206 Multilayer Ceramic Capacitors MLCC - SMD/SMT ROHS"
 			(at 261.62 229.87 0)
 			(effects
@@
 			)
 		)
-		(property "JLCPCB Part #" "C513774"
+		(property "JLCPCB Part #" "C13585"
+			(at 261.62 229.87 0)
+			(effects
+				(font
+					(size 1.27 1.27)
+				)
+				(hide yes)
+			)
+		)
+		(property "Part" "CL31A106KBHNNNE"
 			(at 261.62 229.87 0)
 			(effects
@@
 			)
 		)
-		(property "Description" "-55℃~+125℃ 16V 22uF 350mΩ ±10% 2312 Tantalum Capacitors ROHS"
+		(property "Description" "25V 22uF ±10% CASE-C-6032-28(mm) Tantalum Capacitors ROHS"
 			(at 254 229.87 0)
 			(effects
@@
 			)
 		)
-		(property "Part" "TR3C226K016C0350"
+		(property "Part" "TAJC226K025RNJ"
 			(at 254 229.87 0)
 			(effects
@@
 			)
 		)
-		(property "JLCPCB Part #" "C1954274"
+		(property "JLCPCB Part #" "C7214"
 			(at 254 229.87 0)
 			(effects
@@
 			)
 		)
-		(property "Description" ""
+		(property "Description" "-55℃~+155℃ 150Ω 50V 62.5mW Thick Film Resistor ±1% ±100ppm/℃ 0402 Chip Resistor - Surface Mount ROHS"
 			(at 175.26 226.06 0)
 			(effects
@@
 			)
 		)
-		(property "Description" ""
+		(property "Description" "-55℃~+155℃ 10kΩ 50V 62.5mW Thick Film Resistor ±1% ±100ppm/℃ 0402 Chip Resistor - Surface Mount ROHS"
 			(at 182.88 220.98 0)
 			(effects
@@
 			)
 		)
-		(property "Description" ""
+		(property "Description" "50V 10uF X5R ±10% 1206 Multilayer Ceramic Capacitors MLCC - SMD/SMT ROHS"
 			(at 58.42 36.83 0)
 			(effects
@@
 			)
 		)
-		(property "Part" "CS3216X5R106K500NRI"
+		(property "Part" "CL31A106KBHNNNE"
 			(at 58.42 36.83 0)
 			(effects
@@
 			)
 		)
-		(property "JLCPCB Part #" "C513774"
+		(property "JLCPCB Part #" "C13585"
 			(at 58.42 36.83 0)
 			(effects
@@
 			)
 		)
-		(property "Description" ""
+		(property "Description" "50V 10uF X5R ±10% 1206 Multilayer Ceramic Capacitors MLCC - SMD/SMT ROHS"
 			(at 262.89 44.45 0)
 			(effects
@@
 			)
 		)
-		(property "Part" "CS3216X5R106K500NRI"
+		(property "Part" "CL31A106KBHNNNE"
 			(at 262.89 44.45 0)
 			(effects
@@
 			)
 		)
-		(property "JLCPCB Part #" "C513774"
+		(property "JLCPCB Part #" "C13585"
 			(at 262.89 44.45 0)
 			(effects
@@
 			)
 		)
-		(property "Description" ""
+		(property "Description" "25V 100nF X7R ±5% 0402 Multilayer Ceramic Capacitors MLCC - SMD/SMT ROHS"
 			(at 300.99 231.14 0)
 			(effects
@@
 			)
 		)
-		(property "Description" ""
+		(property "Description" "-55℃~+155℃ 0Ω 75V 100mW Thick Film Resistor ±1% 0603 Chip Resistor - Surface Mount ROHS"
 			(at 330.2 64.77 0)
 			(effects
@@
 			)
 		)
-		(property "Description" ""
+		(property "Description" "25V 100nF X7R ±5% 0402 Multilayer Ceramic Capacitors MLCC - SMD/SMT ROHS"
 			(at 270.51 44.45 0)
 			(effects
@@
 			)
 		)
-		(property "Description" ""
+		(property "Description" "-55℃~+155℃ 4.7kΩ 50V 62.5mW Thick Film Resistor ±1% ±100ppm/℃ 0402 Chip Resistor - Surface Mount ROHS"
 			(at 354.33 57.15 0)
 			(effects
@@
 			)
 		)
-		(property "Description" ""
+		(property "Description" "-55℃~+155℃ 0Ω 75V 100mW Thick Film Resistor ±1% 0603 Chip Resistor - Surface Mount ROHS"
 			(at 351.79 176.53 0)
 			(effects
@@
 			)
 		)
-		(property "Description" ""
+		(property "Description" "-55℃~+155℃ 0Ω 75V 100mW Thick Film Resistor ±1% 0603 Chip Resistor - Surface Mount ROHS"
 			(at 334.01 45.72 0)
 			(effects
@@
 			)
 		)
-		(property "Description" ""
+		(property "Description" "50V 10uF X5R ±10% 1206 Multilayer Ceramic Capacitors MLCC - SMD/SMT ROHS"
 			(at 125.73 24.13 0)
 			(effects
@@
 			)
 		)
-		(property "Part" "CS3216X5R106K500NRI"
+		(property "Part" "CL31A106KBHNNNE"
 			(at 125.73 24.13 0)
 			(effects
@@
 			)
 		)
-		(property "JLCPCB Part #" "C513774"
+		(property "JLCPCB Part #" "C13585"
 			(at 125.73 24.13 0)
 			(effects
@@
 			)
 		)
-		(property "Value" "10nFx50V"
+		(property "Value" "10uFx50V"
 			(at 314.96 232.4163 0)
 			(effects
@@
 			)
 		)
-		(property "Description" ""
+		(property "Description" "50V 10uF X5R ±10% 1206 Multilayer Ceramic Capacitors MLCC - SMD/SMT ROHS"
 			(at 312.42 231.14 0)
 			(effects
@@
 			)
 		)
-		(property "JLCPCB Part #" "C513774"
+		(property "JLCPCB Part #" "C13585"
+			(at 312.42 231.14 0)
+			(effects
+				(font
+					(size 1.27 1.27)
+				)
+				(hide yes)
+			)
+		)
+		(property "Part" "CL31A106KBHNNNE"
 			(at 312.42 231.14 0)
 			(effects
@@
 			)
 		)
-		(property "Description" ""
+		(property "Description" "25V 100nF X7R ±5% 0402 Multilayer Ceramic Capacitors MLCC - SMD/SMT ROHS"
 			(at 120.65 172.72 0)
 			(effects
@@
 			)
 		)
-		(property "Description" ""
+		(property "Description" "25V 100nF X7R ±5% 0402 Multilayer Ceramic Capacitors MLCC - SMD/SMT ROHS"
 			(at 162.56 24.13 0)
 			(effects
@@
 			)
 		)
-		(property "Description" ""
+		(property "Description" "50V 10uF X5R ±10% 1206 Multilayer Ceramic Capacitors MLCC - SMD/SMT ROHS"
 			(at 293.37 231.14 0)
 			(effects
@@
 			)
 		)
-		(property "Part" "CS3216X5R106K500NRI"
+		(property "Part" "CL31A106KBHNNNE"
 			(at 293.37 231.14 0)
 			(effects
@@
 			)
 		)
-		(property "JLCPCB Part #" "C513774"
+		(property "JLCPCB Part #" "C13585"
 			(at 293.37 231.14 0)
 			(effects
@@
 			)
 		)
-		(property "Description" ""
+		(property "Description" "25V 100nF X7R ±5% 0402 Multilayer Ceramic Capacitors MLCC - SMD/SMT ROHS"
 			(at 133.35 24.13 0)
 			(effects
