File: sdio.kicad_sch (KiCad schematic)
At the start: 45 parts, among them IC4 TXS02612RTWR, J23 SCHA1B0100, U30 KLM8G1GETF-B041, U31 AZ1117H-1.8TRE1_SOT223

Commit message: JLCPCB ID attribute updates
These 'JLCPCB Part #' updates reflect the JLCPCB assembly order # SMT026073061946-2250854A
Parts:
- R254: JLCPCB Part # C25900 -> C105871; Part 0402WGF4701TCE -> RC0402FR-074K7L
Changed lines of the file:
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@@
 			)
 		)
-		(property "JLCPCB Part #" "C25900"
+		(property "JLCPCB Part #" "C105871"
 			(at 354.33 57.15 0)
 			(effects
@@
 			)
 		)
-		(property "Part" "0402WGF4701TCE"
+		(property "Part" "RC0402FR-074K7L"
 			(at 354.33 57.15 0)
 			(effects
