File: soc_b0_jtag.kicad_sch (KiCad schematic)
At the start: 37 parts, among them J20 Conn_02x07_Odd_Even, J21 Conn_ARM_SWD_TagConnect_TC2050, J22 Conn_01x02, Q11 BSS138, SW3 SW_Push, U21 XC7Z030_FBG676, U22 SN74LXC1T45DBVR

Commit message: JLCPCB part id's update
Parts:
- R163: JLCPCB Part # C21189 -> C2906974; Part 0603WAF0000T5E -> FRC0603F0000TS
Changed lines of the file:
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@@
 			)
 		)
-		(property "JLCPCB Part #" "C21189"
+		(property "JLCPCB Part #" "C2906974"
 			(at 130.81 257.81 0)
 			(effects
@@
 			)
 		)
-		(property "Part" "0603WAF0000T5E"
+		(property "Part" "FRC0603F0000TS"
 			(at 130.81 257.81 90)
 			(effects
