File: soc_bank500.kicad_sch (KiCad schematic)
At the start: 38 parts, among them SW4 DTS04GE, U21 XC7Z030_FBG676, U23 S25FL128SAGMFI000, U24 TCA6408ARGTR

Commit message: JLCPCB part id's update
Parts:
- R177, R179: JLCPCB Part # C21189 -> C2906974; Part 0603WAF0000T5E -> FRC0603F0000TS
Changed lines of the file:
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@@
 			)
 		)
-		(property "JLCPCB Part #" "C21189"
+		(property "JLCPCB Part #" "C2906974"
 			(at 97.79 50.8 0)
 			(effects
@@
 			)
 		)
-		(property "Part" "0603WAF0000T5E"
+		(property "Part" "FRC0603F0000TS"
 			(at 97.79 50.8 90)
 			(effects
@@
 			)
 		)
-		(property "JLCPCB Part #" "C21189"
-			(at 109.22 48.26 0)
-			(effects
-				(font
-					(size 1.27 1.27)
-				)
-				(hide yes)
-			)
-		)
-		(property "Part" "0603WAF0000T5E"
+		(property "JLCPCB Part #" "C2906974"
+			(at 109.22 48.26 0)
+			(effects
+				(font
+					(size 1.27 1.27)
+				)
+				(hide yes)
+			)
+		)
+		(property "Part" "FRC0603F0000TS"
 			(at 109.22 48.26 90)
 			(effects
