File: soc_bank500.kicad_sch (KiCad schematic)
At the start: 38 parts, among them SW4 DTS04GE, U21 XC7Z030_FBG676, U23 S25FL128SAGMFI000, U24 TCA6408ARGTR

Commit message: bom: substitute out-of-stock passives, sync descriptions to JLCPCB IDs
Every substitution keeps its existing footprint, so no PCB rework is
implied. Stock figures verified against live LCSC, not the parts-library
snapshot (which was stale on four parts).

  C11-C13  C188358 -> C178366   82uF/35V -> 180uF/25V OS-CON SVPF (was OOS)
  R54      C138285 -> C2933137  12.7k 0603 (was OOS)
  31x tant C1954274 -> C7214    22uF 16V -> 25V; ~16 -> ~2580 boards of
                                stock, and fixes the +12VEXT derating on
                                C430/C431 (75% -> 48% of rating)
  20x cap  C513774 -> C13585    10uF 1206, JLC Basic part
  C76,C77  C2918589 -> C541338  4.3pF +-0.1pF, 32.768kHz load caps for Y2
  R286     C705904 -> C2930124  649R, HX2VL RREF
  R45      C2936632 -> C17477   consolidated onto an existing BOM line
  C328     C2170363 -> C368809  consolidated; was outside the JLC library
  R172     C705658 -> C705678   consolidated; was outside the JLC library

Fix eight capacitors labelled 10nFx50V that carried a 10uF part number:
C31 C32 C302 C307 C309 C347 C360 C368 -> value corrected to 10uFx50V.
All sit on power rails or LDO inputs where 10uF is the intent.

Restore C302's Footprint, which had been corrupted to "c9" (not a valid
library reference; would have failed the next PCB update).

Regenerate Description on all 822 R/C from live LCSC parametric data so
each matches its JLCPCB Part #.

Value fields keep the project convention: the voltage suffix is the design
minimum, not the fitted part's rating, so the tantalum stayed 22uFx16V.
C11-C13 did change 82uF -> 180uF because the capacitance itself changed.

Also carries work in progress from this session: H35 mounting hole,
R50/R137/R285 moved to 0402 (C25792), R30 220R -> 330R (C5154013),
C24 -> C1618.

NASR.net and NASR.kicad_pcb still predate these schematic edits; they need
a netlist re-export and Update PCB from Schematic.

Co-Authored-By: Claude Opus 5 (1M context) <noreply@anthropic.c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
Parts:
- R172: JLCPCB Part # C705658 -> C705678; Part RT0402CRD0720KL -> RT0402DRE0720KL
Changed lines of the file:
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@@
 			)
 		)
-		(property "Description" ""
+		(property "Description" "-55℃~+155℃ 10kΩ 50V 62.5mW Thick Film Resistor ±1% ±100ppm/℃ 0402 Chip Resistor - Surface Mount ROHS"
 			(at 91.44 120.65 0)
 			(effects
@@
 			)
 		)
-		(property "Description" ""
+		(property "Description" "-55℃~+155℃ 150Ω 50V 62.5mW Thick Film Resistor ±1% ±100ppm/℃ 0402 Chip Resistor - Surface Mount ROHS"
 			(at 106.68 34.29 0)
 			(effects
@@
 			)
 		)
-		(property "Description" ""
+		(property "Description" "25V 100nF X7R ±5% 0402 Multilayer Ceramic Capacitors MLCC - SMD/SMT ROHS"
 			(at 308.61 185.42 0)
 			(effects
@@
 			)
 		)
-		(property "Description" ""
+		(property "Description" "-55℃~+155℃ 150Ω 50V 62.5mW Thick Film Resistor ±1% ±100ppm/℃ 0402 Chip Resistor - Surface Mount ROHS"
 			(at 242.57 212.09 0)
 			(effects
@@
 			)
 		)
-		(property "Description" ""
+		(property "Description" "-55℃~+155℃ 0Ω 75V 100mW Thick Film Resistor ±1% 0603 Chip Resistor - Surface Mount ROHS"
 			(at 97.79 50.8 0)
 			(effects
@@
 			)
 		)
-		(property "Description" ""
+		(property "Description" "-55℃~+155℃ 0Ω 75V 100mW Thick Film Resistor ±1% 0603 Chip Resistor - Surface Mount ROHS"
 			(at 109.22 48.26 0)
 			(effects
@@
 			)
 		)
-		(property "Description" ""
+		(property "Description" "-55℃~+155℃ 10kΩ 50V 62.5mW Thick Film Resistor ±1% ±100ppm/℃ 0402 Chip Resistor - Surface Mount ROHS"
 			(at 247.65 233.68 0)
 			(effects
@@
 			)
 		)
-		(property "Description" ""
+		(property "Description" "35V 1uF X7R ±10% 0603 Multilayer Ceramic Capacitors MLCC - SMD/SMT ROHS"
 			(at 167.64 92.71 0)
 			(effects
@@
 			)
 		)
-		(property "Description" ""
+		(property "Description" "-55℃~+155℃ 22.1Ω 50V 62.5mW Thick Film Resistor ±1% ±100ppm/℃ 0402 Chip Resistor - Surface Mount ROHS"
 			(at 128.27 27.94 0)
 			(effects
@@
 			)
 		)
-		(property "Description" ""
+		(property "Description" "35V 1uF X7R ±10% 0603 Multilayer Ceramic Capacitors MLCC - SMD/SMT ROHS"
 			(at 190.5 102.87 0)
 			(effects
@@
 			)
 		)
-		(property "Description" ""
+		(property "Description" "-55℃~+155℃ 330Ω 50V 62.5mW Thick Film Resistor ±1% ±100ppm/℃ 0402 Chip Resistor - Surface Mount ROHS"
 			(at 231.14 220.98 0)
 			(effects
@@
 			)
 		)
-		(property "Description" ""
+		(property "Description" "-55℃~+155℃ 20kΩ 50V 62.5mW Thin Film Resistor ±0.5% ±50ppm/℃ 0402 Chip Resistor - Surface Mount ROHS"
 			(at 45.72 200.66 0)
 			(effects
@@
 			)
 		)
-		(property "JLCPCB Part #" "C705658"
+		(property "JLCPCB Part #" "C705678"
 			(at 45.72 200.66 0)
 			(effects
@@
 			)
 		)
-		(property "Part" "RT0402CRD0720KL"
+		(property "Part" "RT0402DRE0720KL"
 			(at 45.72 200.66 0)
 			(effects
@@
 			)
 		)
-		(property "Description" ""
+		(property "Description" "35V 1uF X7R ±10% 0603 Multilayer Ceramic Capacitors MLCC - SMD/SMT ROHS"
 			(at 320.04 185.42 0)
 			(effects

Commit message: bom: substitute out-of-stock semiconductors, fix Y6 case size
Semiconductor sweep (U/IC/Q/D/CR/SW, fan excluded). Stock verified against
live LCSC -- the JLCPCB parts-library snapshot proved unreliable in both
directions, e.g. BAS21 listed as 6 when it actually had 204,880, and the
Zynq listed as 84 when it had 2.

  U40  C411812  -> C164120   PM25LQ010B-SCE (1 in stock) -> W25X10CLSNIG-TR.
                             True drop-in: same 1Mbit density, SOIC-8 150mil,
                             2.3-3.6V, 104MHz, 25-series command set.

  U23  C393875  -> C2959323  S25FL128SAGMFI000 -> S25FL128SAGMFIR00.
                             Model R = SO-16 with RESET# and VIO, which is how
                             pin 3 (FLASH_RST_B) and pin 14 are already wired.
                             On the previous model-0 part both were RFU, so the
                             flash reset had never been functional. Sector type
                             unchanged (0 = uniform 64-KB hybrid), so the U-Boot
                             / MTD layout is unaffected, and Xilinx UG908 Table 44
                             lists s25fl128sxxxxxx0 as supported.

  Y6   C2901601 -> C17326988 SX2M25.000M20F30TNN -> SIT8008BI-21-YYS-25.000000.
                             The old part is a 2520 (2.5x2.0mm) oscillator on an
                             Abracon ASE 3.2x2.5mm land pattern; the new one is a
                             genuine 3225 part, so the existing footprint becomes
                             dimensionally correct. 25MHz +/-20ppm into the
                             LAN8742A reference, well inside the +/-50ppm that
                             100BASE-TX requires. No PCB change.

All three keep their existing footprints, so no re-routing is implied.

Also carries the netlist re-export and PCB sync for the earlier passives work,
which brought schematic, netlist and PCB into agreement across all 826 R/C.

NOTE: NASR.net and NASR.kicad_pcb predate the three substitutions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
Parts:
- U23: value S25FL128SAGMFI000 -> S25FL128SAGMFIR00; JLCPCB Part # C393875 -> C2959323; Part S25FL128SAGMFI000 -> S25FL128SAGMFIR00
Changed lines of the file:
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@@
 			)
 		)
-		(property "Value" "S25FL128SAGMFI000"
+		(property "Value" "S25FL128SAGMFIR00"
 			(at 141.605 93.98 0)
 			(effects
@@
 			)
 		)
-		(property "Description" ""
+		(property "Description" "128Mbit 133MHz 2.7V~3.6V SPI NOR Flash, uniform 64-KB sectors, RESET# and VIO, SOIC-16-300mil ROHS"
 			(at 120.65 100.33 0)
 			(effects
@@
 			)
 		)
-		(property "Part" "S25FL128SAGMFI000"
+		(property "Part" "S25FL128SAGMFIR00"
 			(at 120.65 100.33 0)
 			(effects
@@
 			)
 		)
-		(property "JLCPCB Part #" "C393875"
+		(property "JLCPCB Part #" "C2959323"
 			(at 120.65 100.33 0)
 			(effects
