File: uart.kicad_sch (KiCad schematic)
At the start: 45 parts, among them J17 USB_B, J18 D09P33E4GV00LF, J19 D09P33E4GV00LF, U17 TS5A23159DGS, U18 CP2104, U19 TRS3221ECPW, U20 TRS3221ECPW

Commit message: JLCPCB part id's update
Parts:
- C154, C155, C156, C157, C158, C159, C160, C161: JLCPCB Part # C141172 -> C49678; Part C0805X104K5RACAUTO -> CC0805KRX7R9BB104
- R139, R143, R147, R148, R149, R150: JLCPCB Part # C21189 -> C2906974; Part 0603WAF0000T5E -> FRC0603F0000TS
Changed lines of the file:
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@@
 			)
 		)
-		(property "JLCPCB Part #" "C141172"
+		(property "JLCPCB Part #" "C49678"
 			(at 306.07 54.61 0)
 			(effects
@@
 			)
 		)
-		(property "Part" "C0805X104K5RACAUTO"
+		(property "Part" "CC0805KRX7R9BB104"
 			(at 306.07 54.61 0)
 			(effects
@@
 			)
 		)
-		(property "JLCPCB Part #" "C141172"
+		(property "JLCPCB Part #" "C49678"
 			(at 290.83 46.99 0)
 			(effects
@@
 			)
 		)
-		(property "Part" "C0805X104K5RACAUTO"
+		(property "Part" "CC0805KRX7R9BB104"
 			(at 290.83 46.99 0)
 			(effects
@@
 			)
 		)
-		(property "JLCPCB Part #" "C21189"
+		(property "JLCPCB Part #" "C2906974"
 			(at 351.79 59.69 0)
 			(effects
@@
 			)
 		)
-		(property "Part" "0603WAF0000T5E"
+		(property "Part" "FRC0603F0000TS"
 			(at 351.79 59.69 90)
 			(effects
@@
 			)
 		)
-		(property "JLCPCB Part #" "C21189"
+		(property "JLCPCB Part #" "C2906974"
 			(at 368.3 62.23 0)
 			(effects
@@
 			)
 		)
-		(property "Part" "0603WAF0000T5E"
+		(property "Part" "FRC0603F0000TS"
 			(at 368.3 62.23 90)
 			(effects
@@
 			)
 		)
-		(property "JLCPCB Part #" "C141172"
+		(property "JLCPCB Part #" "C49678"
 			(at 298.45 38.1 0)
 			(effects
@@
 			)
 		)
-		(property "Part" "C0805X104K5RACAUTO"
+		(property "Part" "CC0805KRX7R9BB104"
 			(at 298.45 38.1 0)
 			(effects
@@
 			)
 		)
-		(property "JLCPCB Part #" "C141172"
+		(property "JLCPCB Part #" "C49678"
 			(at 298.45 114.3 0)
 			(effects
@@
 			)
 		)
-		(property "Part" "C0805X104K5RACAUTO"
+		(property "Part" "CC0805KRX7R9BB104"
 			(at 298.45 114.3 0)
 			(effects
@@
 			)
 		)
-		(property "JLCPCB Part #" "C141172"
+		(property "JLCPCB Part #" "C49678"
 			(at 306.07 125.73 0)
 			(effects
@@
 			)
 		)
-		(property "Part" "C0805X104K5RACAUTO"
+		(property "Part" "CC0805KRX7R9BB104"
 			(at 306.07 125.73 0)
 			(effects
@@
 			)
 		)
-		(property "JLCPCB Part #" "C21189"
+		(property "JLCPCB Part #" "C2906974"
 			(at 120.65 50.8 0)
 			(effects
@@
 			)
 		)
-		(property "Part" "0603WAF0000T5E"
+		(property "Part" "FRC0603F0000TS"
 			(at 120.65 50.8 90)
 			(effects
@@
 			)
 		)
-		(property "JLCPCB Part #" "C21189"
+		(property "JLCPCB Part #" "C2906974"
 			(at 107.95 48.26 0)
 			(effects
@@
 			)
 		)
-		(property "Part" "0603WAF0000T5E"
+		(property "Part" "FRC0603F0000TS"
 			(at 107.95 48.26 90)
 			(effects
@@
 			)
 		)
-		(property "JLCPCB Part #" "C141172"
+		(property "JLCPCB Part #" "C49678"
 			(at 306.07 130.81 0)
 			(effects
@@
 			)
 		)
-		(property "Part" "C0805X104K5RACAUTO"
+		(property "Part" "CC0805KRX7R9BB104"
 			(at 306.07 130.81 0)
 			(effects
@@
 			)
 		)
-		(property "JLCPCB Part #" "C141172"
+		(property "JLCPCB Part #" "C49678"
 			(at 306.07 49.53 0)
 			(effects
@@
 			)
 		)
-		(property "Part" "C0805X104K5RACAUTO"
+		(property "Part" "CC0805KRX7R9BB104"
 			(at 306.07 49.53 0)
 			(effects
@@
 			)
 		)
-		(property "JLCPCB Part #" "C21189"
+		(property "JLCPCB Part #" "C2906974"
 			(at 368.3 138.43 0)
 			(effects
@@
 			)
 		)
-		(property "Part" "0603WAF0000T5E"
+		(property "Part" "FRC0603F0000TS"
 			(at 368.3 138.43 90)
 			(effects
@@
 			)
 		)
-		(property "JLCPCB Part #" "C21189"
+		(property "JLCPCB Part #" "C2906974"
 			(at 355.6 135.89 0)
 			(effects
@@
 			)
 		)
-		(property "Part" "0603WAF0000T5E"
+		(property "Part" "FRC0603F0000TS"
 			(at 355.6 135.89 90)
 			(effects
@@
 			)
 		)
-		(property "JLCPCB Part #" "C141172"
+		(property "JLCPCB Part #" "C49678"
 			(at 290.83 123.19 0)
 			(effects
@@
 			)
 		)
-		(property "Part" "C0805X104K5RACAUTO"
+		(property "Part" "CC0805KRX7R9BB104"
 			(at 290.83 123.19 0)
 			(effects
