File: uart.kicad_sch (KiCad schematic)
At the start: 46 parts, among them J17 USB_B, J18 D09P33E4GV00LF, J19 D09P33E4GV00LF, U17 TS5A23159DGS, U18 CP2104, U19 TRS3221ECPW, U20 TRS3221ECPW

Commit message: JLCPCB ID attribute updates
These 'JLCPCB Part #' updates reflect the JLCPCB assembly order # SMT026073061946-2250854A
Parts:
- R138: JLCPCB Part # C25900 -> C105871; Part 0402WGF4701TCE -> RC0402FR-074K7L
Changed lines of the file:
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@@
 			)
 		)
-		(property "JLCPCB Part #" "C25900"
+		(property "JLCPCB Part #" "C105871"
 			(at 68.58 48.26 0)
 			(effects
@@
 			)
 		)
-		(property "Part" "0402WGF4701TCE"
+		(property "Part" "RC0402FR-074K7L"
 			(at 68.58 48.26 0)
 			(effects
