File: usb-hub.kicad_sch (KiCad schematic)
At the start: 43 parts, among them IC5 M24C08-RDW6TP, IC6 CY7C65632-28LTXC, J25 USB_A, U33 CDCLVC1103PW, U34 TXS0102DCT, U35 USB3320C-EZK-TR, X1 X1G0041710018

Commit message: JLCPCB part id's update
Parts:
- R281: JLCPCB Part # C365221 -> C2960681; Part HPCR0603F8K06K9 -> FRC0603F8061TS
Changed lines of the file:
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@@
 			)
 		)
-		(property "JLCPCB Part #" "C365221"
+		(property "JLCPCB Part #" "C2960681"
 			(at 144.78 92.71 0)
 			(effects
@@
 			)
 		)
-		(property "Part" "HPCR0603F8K06K9"
+		(property "Part" "FRC0603F8061TS"
 			(at 144.78 92.71 0)
 			(effects
