File: usb-hub.kicad_sch (KiCad schematic)
At the start: 43 parts, among them IC5 M24C08-RDW6TP, IC6 CY7C65632-28LTXC, J25 USB_A, U33 CDCLVC1103PW, U34 TXS0102DCT, U35 USB3320C-EZK-TR, X1 X1G0041710018

Commit message: minor changes here and there
Parts:
- J25: JLCPCB Part # (none) -> C19944603; Part (none) -> DS1095-WNR0
Changed lines of the file:
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@@
+			)
+		)
+		(property "JLCPCB Part #" "C19944603"
+			(at 229.87 213.36 0)
+			(effects
+				(font
+					(size 1.27 1.27)
+				)
+				(hide yes)
+			)
+		)
+		(property "Part" "DS1095-WNR0"
+			(at 229.87 213.36 0)
+			(effects
+				(font
+					(size 1.27 1.27)
+				)
+				(hide yes)
 			)
 		)
