File: usb-hub.kicad_sch (KiCad schematic)
At the start: 43 parts, among them IC5 M24C08-RDW6TP, IC6 CY7C65632-28LTXC, J25 USB_A, U33 CDCLVC1103PW, U34 TXS0102DCT, U35 USB3320C-EZK-TR, X1 X1G0041710018

Commit message: schema: JTAG connector & resistors, rev change
Parts:
- R287: now not fitted
Changed lines of the file:
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@@
 		(title "NASR-M")
 		(date "2025-10-22")
-		(rev "D 0.9.5")
+		(rev "D 0.9.8")
 		(company "electrodyssey.net")
 		(comment 2 "(c) Nazim 2025")
 		(comment 3 "Author: Nazim Aghabayov")
 		(comment 4 "SYZYGY Carrier Mainboard")
-		(comment 5 "rel: Fletched Bustard")
+		(comment 5 "rel: Wild Goose")
 	)
 	(text "USB_RESET_B\ntranslated to 3V3\nfor a USB HUB Reset"
@@
 		(in_bom yes)
 		(on_board yes)
-		(dnp no)
+		(dnp yes)
 		(property "Reference" "R287"
 			(at 313.182 44.196 90)
