File: usb-hub.kicad_sch (KiCad schematic)
At the start: 43 parts, among them IC5 M24C08-RDW6TP, IC6 CY7C65632-28LTXC, J25 USB_A, U33 CDCLVC1103PW, U34 TXS0102DCT, U35 USB3320C-EZK-TR, X1 X1G0041710018

Commit message: bom: substitute out-of-stock passives, sync descriptions to JLCPCB IDs
Every substitution keeps its existing footprint, so no PCB rework is
implied. Stock figures verified against live LCSC, not the parts-library
snapshot (which was stale on four parts).

  C11-C13  C188358 -> C178366   82uF/35V -> 180uF/25V OS-CON SVPF (was OOS)
  R54      C138285 -> C2933137  12.7k 0603 (was OOS)
  31x tant C1954274 -> C7214    22uF 16V -> 25V; ~16 -> ~2580 boards of
                                stock, and fixes the +12VEXT derating on
                                C430/C431 (75% -> 48% of rating)
  20x cap  C513774 -> C13585    10uF 1206, JLC Basic part
  C76,C77  C2918589 -> C541338  4.3pF +-0.1pF, 32.768kHz load caps for Y2
  R286     C705904 -> C2930124  649R, HX2VL RREF
  R45      C2936632 -> C17477   consolidated onto an existing BOM line
  C328     C2170363 -> C368809  consolidated; was outside the JLC library
  R172     C705658 -> C705678   consolidated; was outside the JLC library

Fix eight capacitors labelled 10nFx50V that carried a 10uF part number:
C31 C32 C302 C307 C309 C347 C360 C368 -> value corrected to 10uFx50V.
All sit on power rails or LDO inputs where 10uF is the intent.

Restore C302's Footprint, which had been corrupted to "c9" (not a valid
library reference; would have failed the next PCB update).

Regenerate Description on all 822 R/C from live LCSC parametric data so
each matches its JLCPCB Part #.

Value fields keep the project convention: the voltage suffix is the design
minimum, not the fitted part's rating, so the tantalum stayed 22uFx16V.
C11-C13 did change 82uF -> 180uF because the capacitance itself changed.

Also carries work in progress from this session: H35 mounting hole,
R50/R137/R285 moved to 0402 (C25792), R30 220R -> 330R (C5154013),
C24 -> C1618.

NASR.net and NASR.kicad_pcb still predate these schematic edits; they need
a netlist re-export and Update PCB from Schematic.

Co-Authored-By: Claude Opus 5 (1M context) <noreply@anthropic.c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
Parts:
- C345, C346: JLCPCB Part # C1954274 -> C7214; Part TR3C226K016C0350 -> TAJC226K025RNJ
- C347: value 10nFx50V -> 10uFx50V; JLCPCB Part # C513774 -> C13585; Part (none) -> CL31A106KBHNNNE
- R285: footprint Resistor_SMD:R_0603_1608Metric -> Resistor_SMD:R_0402_1005Metric; JLCPCB Part # C5139555 -> C25792; Part (none) -> 0402WGF4702TCE
- R286: JLCPCB Part # C705904 -> C2930124; Part RT0603CRD07649RL -> FRC0603F6490TS
Changed lines of the file:
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@@
 			)
 		)
-		(property "Description" ""
+		(property "Description" "50V 10nF X7R ±10% 0805 Multilayer Ceramic Capacitors MLCC - SMD/SMT ROHS"
 			(at 38.1 147.32 0)
 			(effects
@@
 			)
 		)
-		(property "Description" "-55℃~+125℃ 16V 22uF 350mΩ ±10% 2312 Tantalum Capacitors ROHS"
+		(property "Description" "25V 22uF ±10% CASE-C-6032-28(mm) Tantalum Capacitors ROHS"
 			(at 198.12 185.42 0)
 			(effects
@@
 			)
 		)
-		(property "Part" "TR3C226K016C0350"
+		(property "Part" "TAJC226K025RNJ"
 			(at 198.12 185.42 0)
 			(effects
@@
 			)
 		)
-		(property "JLCPCB Part #" "C1954274"
+		(property "JLCPCB Part #" "C7214"
 			(at 198.12 185.42 0)
 			(effects
@@
 			)
 		)
-		(property "Description" ""
+		(property "Description" "25V 100nF X7R ±5% 0402 Multilayer Ceramic Capacitors MLCC - SMD/SMT ROHS"
 			(at 299.72 26.67 0)
 			(effects
@@
 			)
 		)
-		(property "Description" ""
+		(property "Description" "-55℃~+155℃ 4.7kΩ 50V 62.5mW Thick Film Resistor ±1% ±100ppm/℃ 0402 Chip Resistor - Surface Mount ROHS"
 			(at 264.16 100.33 0)
 			(effects
@@
 			)
 		)
-		(property "Description" ""
+		(property "Description" "25V 100nF X7R ±5% 0402 Multilayer Ceramic Capacitors MLCC - SMD/SMT ROHS"
 			(at 251.46 39.37 0)
 			(effects
@@
 			)
 		)
-		(property "Footprint" "Resistor_SMD:R_0603_1608Metric"
+		(property "Footprint" "Resistor_SMD:R_0402_1005Metric"
 			(at 264.16 116.84 0)
 			(effects
@@
 			)
 		)
-		(property "Description" ""
+		(property "Description" "-55℃~+155℃ 47kΩ 50V 62.5mW Thick Film Resistor ±1% ±100ppm/℃ 0402 Chip Resistor - Surface Mount ROHS"
 			(at 264.16 116.84 0)
 			(effects
@@
 			)
 		)
-		(property "JLCPCB Part #" "C5139555"
+		(property "JLCPCB Part #" "C25792"
 			(at 264.16 116.84 0)
 			(effects
@@
 			)
 		)
+		(property "Part" "0402WGF4702TCE"
+			(at 264.16 116.84 0)
+			(effects
+				(font
+					(size 1.27 1.27)
+				)
+				(hide yes)
+			)
+		)
 		(pin "2"
 		)
@@
 			)
 		)
-		(property "Description" ""
+		(property "Description" "25V 100nF X7R ±5% 0402 Multilayer Ceramic Capacitors MLCC - SMD/SMT ROHS"
 			(at 27.94 246.38 0)
 			(effects
@@
 			)
 		)
-		(property "Description" ""
+		(property "Description" "35V 1uF X7R ±10% 0603 Multilayer Ceramic Capacitors MLCC - SMD/SMT ROHS"
 			(at 264.16 40.64 0)
 			(effects
@@
 			)
 		)
-		(property "Description" ""
+		(property "Description" "35V 1uF X7R ±10% 0603 Multilayer Ceramic Capacitors MLCC - SMD/SMT ROHS"
 			(at 53.34 195.58 0)
 			(effects
@@
 			)
 		)
-		(property "Description" ""
+		(property "Description" "-55℃~+155℃ 8.06kΩ 75V 100mW Thick Film Resistor ±1% ±100ppm/℃ 0603 Chip Resistor - Surface Mount ROHS"
 			(at 144.78 92.71 0)
 			(effects
@@
 			)
 		)
-		(property "Description" ""
+		(property "Description" "35V 1uF X7R ±10% 0603 Multilayer Ceramic Capacitors MLCC - SMD/SMT ROHS"
 			(at 93.98 238.76 0)
 			(effects
@@
 			)
 		)
-		(property "Description" ""
+		(property "Description" "-55℃~+155℃ 10kΩ 50V 62.5mW Thick Film Resistor ±1% ±100ppm/℃ 0402 Chip Resistor - Surface Mount ROHS"
 			(at 119.38 71.12 0)
 			(effects
@@
 			)
 		)
-		(property "Description" ""
+		(property "Description" "25V 100nF X7R ±5% 0402 Multilayer Ceramic Capacitors MLCC - SMD/SMT ROHS"
 			(at 38.1 229.87 0)
 			(effects
@@
 			)
 		)
-		(property "Description" ""
+		(property "Description" "35V 1uF X7R ±10% 0603 Multilayer Ceramic Capacitors MLCC - SMD/SMT ROHS"
 			(at 312.42 26.67 0)
 			(effects
@@
 			)
 		)
-		(property "Description" ""
+		(property "Description" "-55℃~+155℃ 10kΩ 50V 62.5mW Thick Film Resistor ±1% ±100ppm/℃ 0402 Chip Resistor - Surface Mount ROHS"
 			(at 257.81 105.41 0)
 			(effects
@@
 			)
 		)
-		(property "Description" ""
+		(property "Description" "50V 10nF X7R ±10% 0805 Multilayer Ceramic Capacitors MLCC - SMD/SMT ROHS"
 			(at 41.91 195.58 0)
 			(effects
@@
 			)
 		)
-		(property "Description" ""
+		(property "Description" "25V 100nF X7R ±5% 0402 Multilayer Ceramic Capacitors MLCC - SMD/SMT ROHS"
 			(at 74.93 86.36 0)
 			(effects
@@
 			)
 		)
-		(property "Description" ""
+		(property "Description" "35V 1uF X7R ±10% 0603 Multilayer Ceramic Capacitors MLCC - SMD/SMT ROHS"
 			(at 39.37 246.38 0)
 			(effects
@@
 			)
 		)
-		(property "Description" "-55℃~+125℃ 16V 22uF 350mΩ ±10% 2312 Tantalum Capacitors ROHS"
+		(property "Description" "25V 22uF ±10% CASE-C-6032-28(mm) Tantalum Capacitors ROHS"
 			(at 209.55 185.42 0)
 			(effects
@@
 			)
 		)
-		(property "Part" "TR3C226K016C0350"
+		(property "Part" "TAJC226K025RNJ"
 			(at 209.55 185.42 0)
 			(effects
@@
 			)
 		)
-		(property "JLCPCB Part #" "C1954274"
+		(property "JLCPCB Part #" "C7214"
 			(at 209.55 185.42 0)
 			(effects
@@
 			)
 		)
-		(property "Description" ""
+		(property "Description" "25V 100nF X7R ±5% 0402 Multilayer Ceramic Capacitors MLCC - SMD/SMT ROHS"
 			(at 72.39 219.71 0)
 			(effects
@@
 			)
 		)
-		(property "Description" ""
+		(property "Description" "-55℃~+155℃ 4.7kΩ 50V 62.5mW Thick Film Resistor ±1% ±100ppm/℃ 0402 Chip Resistor - Surface Mount ROHS"
 			(at 52.07 100.33 0)
 			(effects
@@
 			)
 		)
-		(property "Description" ""
+		(property "Description" "35V 1uF X7R ±10% 0603 Multilayer Ceramic Capacitors MLCC - SMD/SMT ROHS"
 			(at 273.05 116.84 0)
 			(effects
@@
 			)
 		)
-		(property "Description" ""
+		(property "Description" "35V 1uF X7R ±10% 0603 Multilayer Ceramic Capacitors MLCC - SMD/SMT ROHS"
 			(at 83.82 219.71 0)
 			(effects
@@
 			)
 		)
-		(property "Description" ""
+		(property "Description" "-55℃~+155℃ 40.2Ω 50V 62.5mW Thin Film Resistor ±1% ±50ppm/℃ 0402 Chip Resistor - Surface Mount ROHS"
 			(at 111.76 38.1 0)
 			(effects
@@
 			)
 		)
-		(property "Description" ""
+		(property "Description" "-55℃~+155℃ 200kΩ 75V 100mW Thin Film Resistor ±0.1% ±25ppm/℃ 0603 Chip Resistor - Surface Mount ROHS"
 			(at 312.42 48.26 0)
 			(effects
@@
 			)
 		)
-		(property "Description" ""
+		(property "Description" "25V 100nF X7R ±5% 0402 Multilayer Ceramic Capacitors MLCC - SMD/SMT ROHS"
 			(at 226.06 86.36 0)
 			(effects
@@
 			)
 		)
-		(property "Description" ""
+		(property "Description" "-55℃~+155℃ 40.2Ω 50V 62.5mW Thin Film Resistor ±1% ±50ppm/℃ 0402 Chip Resistor - Surface Mount ROHS"
 			(at 262.89 64.77 0)
 			(effects
@@
 			)
 		)
-		(property "Value" "10nFx50V"
+		(property "Value" "10uFx50V"
 			(at 223.52 186.6963 0)
 			(effects
@@
 			)
 		)
-		(property "Description" ""
+		(property "Description" "50V 10uF X5R ±10% 1206 Multilayer Ceramic Capacitors MLCC - SMD/SMT ROHS"
 			(at 220.98 185.42 0)
 			(effects
@@
 			)
 		)
-		(property "JLCPCB Part #" "C513774"
+		(property "JLCPCB Part #" "C13585"
+			(at 220.98 185.42 0)
+			(effects
+				(font
+					(size 1.27 1.27)
+				)
+				(hide yes)
+			)
+		)
+		(property "Part" "CL31A106KBHNNNE"
 			(at 220.98 185.42 0)
 			(effects
@@
 			)
 		)
-		(property "Description" ""
+		(property "Description" "-55℃~+155℃ 649Ω 75V 100mW Thick Film Resistor ±1% ±100ppm/℃ 0603 Chip Resistor - Surface Mount ROHS"
 			(at 288.29 118.11 0)
 			(effects
@@
 			)
 		)
-		(property "JLCPCB Part #" "C705904"
+		(property "JLCPCB Part #" "C2930124"
 			(at 288.29 118.11 0)
 			(effects
@@
 			)
 		)
-		(property "Part" "RT0603CRD07649RL"
+		(property "Part" "FRC0603F6490TS"
 			(at 288.29 118.11 90)
 			(effects
@@
 			)
 		)
-		(property "Description" ""
+		(property "Description" "-55℃~+155℃ 150Ω 50V 62.5mW Thick Film Resistor ±1% ±100ppm/℃ 0402 Chip Resistor - Surface Mount ROHS"
 			(at 20.32 163.83 0)
 			(effects
@@
 			)
 		)
-		(property "Description" ""
+		(property "Description" "25V 100nF X7R ±5% 0402 Multilayer Ceramic Capacitors MLCC - SMD/SMT ROHS"
 			(at 58.42 86.36 0)
 			(effects
