File: usb-hub.kicad_sch (KiCad schematic)
At the start: 43 parts, among them IC5 M24C08-RDW6TP, IC6 CY7C65632-28LTXC, J25 USB_A, U33 CDCLVC1103PW, U34 TXS0102DCT, U35 USB3320C-EZK-TR, X1 X1G0041710018

Commit message: JLCPCB ID attribute updates
These 'JLCPCB Part #' updates reflect the JLCPCB assembly order # SMT026073061946-2250854A
Parts:
- R278, R284: JLCPCB Part # C25900 -> C105871; Part 0402WGF4701TCE -> RC0402FR-074K7L
Changed lines of the file:
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@@
 			)
 		)
-		(property "JLCPCB Part #" "C25900"
+		(property "JLCPCB Part #" "C105871"
 			(at 264.16 100.33 0)
 			(effects
@@
 			)
 		)
-		(property "Part" "0402WGF4701TCE"
+		(property "Part" "RC0402FR-074K7L"
 			(at 264.16 100.33 0)
 			(effects
@@
 			)
 		)
-		(property "JLCPCB Part #" "C25900"
+		(property "JLCPCB Part #" "C105871"
 			(at 52.07 100.33 0)
 			(effects
@@
 			)
 		)
-		(property "Part" "0402WGF4701TCE"
+		(property "Part" "RC0402FR-074K7L"
 			(at 52.07 100.33 0)
 			(effects
