File: usb-sata.kicad_sch (KiCad schematic)
At the start: 52 parts, among them IC7 TPS74611PQWDRVRQ1, J26 TagConnect_TC2050, J27 292161-3, J28 MDT420M02001, U36 TUSB9261IPVP, U37 TLV71311PDBV, U38 AZ1117-3.3, U39 AZ1117-3.3, U40 PM25LQ010B-SCE, Y5 ECS-TXO-32CSMV-400-BN-TR

Commit message: JLCPCB part id's update
Parts:
- FB35: value GZ1608D601TF -> BLM18AG601SN1D; JLCPCB Part # C1002 -> C19330; Part GZ1608D601TF -> BLM18AG601SN1D
- R288, R295, R300, R301: JLCPCB Part # C2936632 -> C17477; Part (none) -> 0805W8F0000T5E
Changed lines of the file:
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@@
 			)
 		)
-		(property "Value" "GZ1608D601TF"
+		(property "Value" "BLM18AG601SN1D"
 			(at 177.8 25.438 0)
 			(effects
@@
 			)
 		)
-		(property "JLCPCB Part #" "C1002"
+		(property "JLCPCB Part #" "C19330"
 			(at 175.26 24.13 0)
 			(effects
@@
 			)
 		)
-		(property "Part" "GZ1608D601TF"
+		(property "Part" "BLM18AG601SN1D"
 			(at 175.26 24.13 90)
 			(effects
@@
 			)
 		)
-		(property "JLCPCB Part #" "C2936632"
+		(property "JLCPCB Part #" "C17477"
 			(at 223.52 100.33 0)
 			(effects
@@
 			)
 		)
+		(property "Part" "0805W8F0000T5E"
+			(at 223.52 100.33 90)
+			(effects
+				(font
+					(size 1.27 1.27)
+				)
+				(hide yes)
+			)
+		)
 		(pin "2"
 		)
@@
 			)
 		)
-		(property "JLCPCB Part #" "C2936632"
+		(property "JLCPCB Part #" "C17477"
 			(at 137.16 248.92 0)
 			(effects
@@
 			)
 		)
+		(property "Part" "0805W8F0000T5E"
+			(at 137.16 248.92 0)
+			(effects
+				(font
+					(size 1.27 1.27)
+				)
+				(hide yes)
+			)
+		)
 		(pin "2"
 		)
@@
 			)
 		)
-		(property "JLCPCB Part #" "C2936632"
+		(property "JLCPCB Part #" "C17477"
 			(at 20.32 251.46 0)
 			(effects
@@
 			)
 		)
+		(property "Part" "0805W8F0000T5E"
+			(at 20.32 251.46 0)
+			(effects
+				(font
+					(size 1.27 1.27)
+				)
+				(hide yes)
+			)
+		)
 		(pin "2"
 		)
@@
 			)
 		)
-		(property "JLCPCB Part #" "C2936632"
+		(property "JLCPCB Part #" "C17477"
 			(at 224.79 242.57 0)
 			(effects
@@
 			(at 224.79 242.57 0)
 			(effects
+				(font
+					(size 1.27 1.27)
+				)
+				(hide yes)
+			)
+		)
+		(property "Part" "0805W8F0000T5E"
+			(at 224.79 242.57 0)
+			(effects
