File: usb-sata.kicad_sch (KiCad schematic)
At the start: 52 parts, among them IC7 TPS74611PQWDRVRQ1, J26 TagConnect_TC2050, J27 292161-3, J28 MDT420M02001, U36 TUSB9261IPVP, U37 TLV71311PDBV, U38 AZ1117-3.3, U39 AZ1117-3.3, U40 PM25LQ010B-SCE, Y5 ECS-TXO-32CSMV-400-BN-TR

Commit message: schema: JTAG connector & resistors, rev change
Parts:
- R294, R297, R298: value 100 -> 150; JLCPCB Part # C153111 -> C25082; Part RM04FTN1000 -> 0402WGF1500TCE
Connections:
- no-connect marks 61 -> 62
Changed lines of the file:
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@@
 		(title "NASR-M")
 		(date "2025-10-22")
-		(rev "D 0.9.5")
+		(rev "D 0.9.8")
 		(company "electrodyssey.net")
 		(comment 1 "USB to SATA converter")
@@
 		(comment 3 "Author: Nazim Aghabayov")
 		(comment 4 "SYZYGY Carrier Mainboard")
-		(comment 5 "rel: Fletched Bustard")
+		(comment 5 "rel: Wild Goose")
 	)
 	(bus_alias "USB_D_BUS"
@@
 	)
 	(no_connect
+		(at 73.66 100.33)
+	)
+	(no_connect
 		(at 35.56 132.08)
 	)
@@
 	)
 	(no_connect
+		(at 55.88 100.33)
+	)
+	(no_connect
 		(at 69.85 267.97)
 	)
@@
 		(at 351.79 119.38)
 	)
-	(no_connect
-		(at 55.88 99.06)
-	)
 	(bus_entry
 		(at 138.43 152.4)
@@
 	(wire
 		(pts
-			(xy 55.88 101.6) (xy 53.34 101.6)
+			(xy 55.88 102.87) (xy 53.34 102.87)
 		)
 		(stroke
@@
 	(wire
 		(pts
-			(xy 53.34 101.6) (xy 53.34 104.14)
+			(xy 53.34 102.87) (xy 53.34 104.14)
 		)
 		(stroke
@@
 			)
 		)
-		(property "Value" "100"
+		(property "Value" "150"
 			(at 162.052 116.84 90)
 			(effects
@@
 			)
 		)
-		(property "JLCPCB Part #" "C153111"
+		(property "JLCPCB Part #" "C25082"
 			(at 157.48 118.11 0)
 			(effects
@@
 			)
 		)
-		(property "Part" "RM04FTN1000"
+		(property "Part" "0402WGF1500TCE"
 			(at 157.48 118.11 90)
 			(effects
@@
 		(pin "4"
 		)
+		(pin "9"
+		)
 		(instances
 			(project "NASR"
@@
 			)
 		)
-		(property "Value" "100"
+		(property "Value" "150"
 			(at 163.322 198.12 90)
 			(effects
@@
 			)
 		)
-		(property "JLCPCB Part #" "C153111"
+		(property "JLCPCB Part #" "C25082"
 			(at 158.75 199.39 0)
 			(effects
@@
 			)
 		)
-		(property "Part" "RM04FTN1000"
+		(property "Part" "0402WGF1500TCE"
 			(at 158.75 199.39 90)
 			(effects
@@
 			)
 		)
-		(property "Value" "100"
+		(property "Value" "150"
 			(at 117.602 204.47 90)
 			(effects
@@
 			)
 		)
-		(property "JLCPCB Part #" "C153111"
+		(property "JLCPCB Part #" "C25082"
 			(at 113.03 205.74 0)
 			(effects
@@
 			)
 		)
-		(property "Part" "RM04FTN1000"
+		(property "Part" "0402WGF1500TCE"
 			(at 113.03 205.74 90)
 			(effects
