File: usb-sata.kicad_sch (KiCad schematic)
At the start: 52 parts, among them IC7 TPS74611PQWDRVRQ1, J26 TagConnect_TC2050, J27 292161-3, J28 MDT420M02001, U36 TUSB9261IPVP, U37 TLV71311PDBV, U38 AZ1117-3.3, U39 AZ1117-3.3, U40 PM25LQ010B-SCE, Y5 ECS-TXO-32CSMV-400-BN-TR

Commit message: bom: substitute out-of-stock passives, sync descriptions to JLCPCB IDs
Every substitution keeps its existing footprint, so no PCB rework is
implied. Stock figures verified against live LCSC, not the parts-library
snapshot (which was stale on four parts).

  C11-C13  C188358 -> C178366   82uF/35V -> 180uF/25V OS-CON SVPF (was OOS)
  R54      C138285 -> C2933137  12.7k 0603 (was OOS)
  31x tant C1954274 -> C7214    22uF 16V -> 25V; ~16 -> ~2580 boards of
                                stock, and fixes the +12VEXT derating on
                                C430/C431 (75% -> 48% of rating)
  20x cap  C513774 -> C13585    10uF 1206, JLC Basic part
  C76,C77  C2918589 -> C541338  4.3pF +-0.1pF, 32.768kHz load caps for Y2
  R286     C705904 -> C2930124  649R, HX2VL RREF
  R45      C2936632 -> C17477   consolidated onto an existing BOM line
  C328     C2170363 -> C368809  consolidated; was outside the JLC library
  R172     C705658 -> C705678   consolidated; was outside the JLC library

Fix eight capacitors labelled 10nFx50V that carried a 10uF part number:
C31 C32 C302 C307 C309 C347 C360 C368 -> value corrected to 10uFx50V.
All sit on power rails or LDO inputs where 10uF is the intent.

Restore C302's Footprint, which had been corrupted to "c9" (not a valid
library reference; would have failed the next PCB update).

Regenerate Description on all 822 R/C from live LCSC parametric data so
each matches its JLCPCB Part #.

Value fields keep the project convention: the voltage suffix is the design
minimum, not the fitted part's rating, so the tantalum stayed 22uFx16V.
C11-C13 did change 82uF -> 180uF because the capacitance itself changed.

Also carries work in progress from this session: H35 mounting hole,
R50/R137/R285 moved to 0402 (C25792), R30 220R -> 330R (C5154013),
C24 -> C1618.

NASR.net and NASR.kicad_pcb still predate these schematic edits; they need
a netlist re-export and Update PCB from Schematic.

Co-Authored-By: Claude Opus 5 (1M context) <noreply@anthropic.c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
Parts:
- C358, C359, C362, C366, C367, C369: JLCPCB Part # C1954274 -> C7214; Part TR3C226K016C0350 -> TAJC226K025RNJ
- C360, C368: value 10nFx50V -> 10uFx50V; JLCPCB Part # C513774 -> C13585; Part (none) -> CL31A106KBHNNNE

Commit message: bom: substitute out-of-stock semiconductors, fix Y6 case size
Semiconductor sweep (U/IC/Q/D/CR/SW, fan excluded). Stock verified against
live LCSC -- the JLCPCB parts-library snapshot proved unreliable in both
directions, e.g. BAS21 listed as 6 when it actually had 204,880, and the
Zynq listed as 84 when it had 2.

  U40  C411812  -> C164120   PM25LQ010B-SCE (1 in stock) -> W25X10CLSNIG-TR.
                             True drop-in: same 1Mbit density, SOIC-8 150mil,
                             2.3-3.6V, 104MHz, 25-series command set.

  U23  C393875  -> C2959323  S25FL128SAGMFI000 -> S25FL128SAGMFIR00.
                             Model R = SO-16 with RESET# and VIO, which is how
                             pin 3 (FLASH_RST_B) and pin 14 are already wired.
                             On the previous model-0 part both were RFU, so the
                             flash reset had never been functional. Sector type
                             unchanged (0 = uniform 64-KB hybrid), so the U-Boot
                             / MTD layout is unaffected, and Xilinx UG908 Table 44
                             lists s25fl128sxxxxxx0 as supported.

  Y6   C2901601 -> C17326988 SX2M25.000M20F30TNN -> SIT8008BI-21-YYS-25.000000.
                             The old part is a 2520 (2.5x2.0mm) oscillator on an
                             Abracon ASE 3.2x2.5mm land pattern; the new one is a
                             genuine 3225 part, so the existing footprint becomes
                             dimensionally correct. 25MHz +/-20ppm into the
                             LAN8742A reference, well inside the +/-50ppm that
                             100BASE-TX requires. No PCB change.

All three keep their existing footprints, so no re-routing is implied.

Also carries the netlist re-export and PCB sync for the earlier passives work,
which brought schematic, netlist and PCB into agreement across all 826 R/C.

NOTE: NASR.net and NASR.kicad_pcb predate the three substitutions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
Parts:
- U40: value PM25LQ010B-SCE -> W25X10CLSNIG; JLCPCB Part # C411812 -> C164120; Part (none) -> W25X10CLSNIG-TR
Changed lines of the file:
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@@
 			)
 		)
-		(property "Value" "PM25LQ010B-SCE"
+		(property "Value" "W25X10CLSNIG"
 			(at 261.62 87.63 0)
 			(effects
@@
 			)
 		)
-		(property "JLCPCB Part #" "C411812"
+		(property "JLCPCB Part #" "C164120"
 			(at 261.62 100.33 0)
 			(effects
+				(font
+					(size 1.27 1.27)
+				)
+				(hide yes)
+			)
+		)
+		(property "Part" "W25X10CLSNIG-TR"
+			(at 261.62 100.33 0)
+			(effects
