File: usb-sata.kicad_sch (KiCad schematic)
At the start: 52 parts, among them IC7 TPS74611PQWDRVRQ1, J26 TagConnect_TC2050, J27 292161-3, J28 MDT420M02001, U36 TUSB9261IPVP, U37 TLV71311PDBV, U38 AZ1117-3.3, U39 AZ1117-3.3, U40 W25X10CLSNIG, Y5 ECS-TXO-32CSMV-400-BN-TR

Commit message: MCU TagConnect nRST, SATA socket
MCU TagConnect now connects to NRST net of the MCU.
SATA socket is not DNP any more
Parts:
- J28: now fitted
Changed lines of the file:
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@@
 		(in_bom yes)
 		(on_board yes)
-		(dnp yes)
+		(dnp no)
 		(fields_autoplaced yes)
 		(property "Reference" "J28"

Commit message: JLCPCB ID attribute updates
These 'JLCPCB Part #' updates reflect the JLCPCB assembly order # SMT026073061946-2250854A
Parts:
- R289, R290, R291, R292: JLCPCB Part # C25900 -> C105871; Part 0402WGF4701TCE -> RC0402FR-074K7L
Changed lines of the file:
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@@
 			)
 		)
-		(property "JLCPCB Part #" "C25900"
+		(property "JLCPCB Part #" "C105871"
 			(at 72.39 25.4 0)
 			(effects
@@
 			)
 		)
-		(property "Part" "0402WGF4701TCE"
+		(property "Part" "RC0402FR-074K7L"
 			(at 72.39 25.4 0)
 			(effects
@@
 			)
 		)
-		(property "JLCPCB Part #" "C25900"
+		(property "JLCPCB Part #" "C105871"
 			(at 72.39 33.02 0)
 			(effects
@@
 			)
 		)
-		(property "Part" "0402WGF4701TCE"
+		(property "Part" "RC0402FR-074K7L"
 			(at 72.39 33.02 0)
 			(effects
@@
 			)
 		)
-		(property "JLCPCB Part #" "C25900"
+		(property "JLCPCB Part #" "C105871"
 			(at 30.48 33.02 0)
 			(effects
@@
 			)
 		)
-		(property "Part" "0402WGF4701TCE"
+		(property "Part" "RC0402FR-074K7L"
 			(at 30.48 33.02 0)
 			(effects
@@
 			)
 		)
-		(property "JLCPCB Part #" "C25900"
+		(property "JLCPCB Part #" "C105871"
 			(at 30.48 25.4 0)
 			(effects
@@
 			)
 		)
-		(property "Part" "0402WGF4701TCE"
+		(property "Part" "RC0402FR-074K7L"
 			(at 30.48 25.4 0)
 			(effects
