File: vio_power.kicad_sch (KiCad schematic)
At the start: 55 parts, among them J29 292161-3, U41 TCA6408ARGTR, U42 AZ1117H-1.8TRE1_SOT223, U43 LP2985-3.3, U44 MCP4728, U45 TPS7A4501DCQR, U46 TPS7A4501DCQR

Commit message: JLCPCB part id's update
Parts:
- R319, R320: JLCPCB Part # C2936632 -> C17477; Part (none) -> 0805W8F0000T5E
Changed lines of the file:
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@@
 			)
 		)
-		(property "JLCPCB Part #" "C2936632"
+		(property "JLCPCB Part #" "C17477"
 			(at 154.94 241.3 0)
 			(effects
@@
 		)
 		(property "Mouser " ""
+			(at 154.94 241.3 0)
+			(effects
+				(font
+					(size 1.27 1.27)
+				)
+				(hide yes)
+			)
+		)
+		(property "Part" "0805W8F0000T5E"
 			(at 154.94 241.3 0)
 			(effects
@@
 			)
 		)
-		(property "JLCPCB Part #" "C2936632"
+		(property "JLCPCB Part #" "C17477"
 			(at 154.94 170.18 0)
 			(effects
@@
 			(at 154.94 170.18 0)
 			(effects
+				(font
+					(size 1.27 1.27)
+				)
+				(hide yes)
+			)
+		)
+		(property "Part" "0805W8F0000T5E"
+			(at 154.94 170.18 0)
+			(effects
