File: psddr3.kicad_sch (KiCad schematic)
At the start: 103 parts, among them U21 XC7Z030_FBG676, U27 MT41K256M16TW-107:P, U28 TPS51200DRC, U29 MT41K256M16TW-107:P

Commit message: jlcpcb id's update
Parts:
- C234, C237, C241, C245, C248, C255, C257, C260, C262, C266, C268, C271, C277, C280, C282, C284, C286, C288, C290, C292: JLCPCB Part # C338031 -> C285010; Part C0603X5R1A103KT00NN -> 0201B103K250NT
Changed lines of the file:
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@@
 			)
 		)
-		(property "JLCPCB Part #" "C338031"
+		(property "JLCPCB Part #" "C285010"
 			(at 168.91 148.59 0)
 			(effects
@@
 			)
 		)
-		(property "Part" "C0603X5R1A103KT00NN"
+		(property "Part" "0201B103K250NT"
 			(at 168.91 148.59 0)
 			(effects
@@
 			)
 		)
-		(property "JLCPCB Part #" "C338031"
+		(property "JLCPCB Part #" "C285010"
 			(at 381 147.32 0)
 			(effects
@@
 			)
 		)
-		(property "Part" "C0603X5R1A103KT00NN"
+		(property "Part" "0201B103K250NT"
 			(at 381 147.32 0)
 			(effects
@@
 			)
 		)
-		(property "JLCPCB Part #" "C338031"
+		(property "JLCPCB Part #" "C285010"
 			(at 158.75 148.59 0)
 			(effects
@@
 			)
 		)
-		(property "Part" "C0603X5R1A103KT00NN"
+		(property "Part" "0201B103K250NT"
 			(at 158.75 148.59 0)
 			(effects
@@
 			)
 		)
-		(property "JLCPCB Part #" "C338031"
+		(property "JLCPCB Part #" "C285010"
 			(at 391.16 147.32 0)
 			(effects
@@
 			)
 		)
-		(property "Part" "C0603X5R1A103KT00NN"
+		(property "Part" "0201B103K250NT"
 			(at 391.16 147.32 0)
 			(effects
@@
 			)
 		)
-		(property "JLCPCB Part #" "C338031"
+		(property "JLCPCB Part #" "C285010"
 			(at 370.84 147.32 0)
 			(effects
@@
 			)
 		)
-		(property "Part" "C0603X5R1A103KT00NN"
+		(property "Part" "0201B103K250NT"
 			(at 370.84 147.32 0)
 			(effects
@@
 			)
 		)
-		(property "JLCPCB Part #" "C338031"
+		(property "JLCPCB Part #" "C285010"
 			(at 274.32 149.86 0)
 			(effects
@@
 			)
 		)
-		(property "Part" "C0603X5R1A103KT00NN"
+		(property "Part" "0201B103K250NT"
 			(at 274.32 149.86 0)
 			(effects
@@
 			)
 		)
-		(property "JLCPCB Part #" "C338031"
+		(property "JLCPCB Part #" "C285010"
 			(at 243.84 147.32 0)
 			(effects
@@
 			)
 		)
-		(property "Part" "C0603X5R1A103KT00NN"
+		(property "Part" "0201B103K250NT"
 			(at 243.84 147.32 0)
 			(effects
@@
 			)
 		)
-		(property "JLCPCB Part #" "C338031"
+		(property "JLCPCB Part #" "C285010"
 			(at 285.75 149.86 0)
 			(effects
@@
 			)
 		)
-		(property "Part" "C0603X5R1A103KT00NN"
+		(property "Part" "0201B103K250NT"
 			(at 285.75 149.86 0)
 			(effects
@@
 			)
 		)
-		(property "JLCPCB Part #" "C338031"
+		(property "JLCPCB Part #" "C285010"
 			(at 148.59 148.59 0)
 			(effects
@@
 			)
 		)
-		(property "Part" "C0603X5R1A103KT00NN"
+		(property "Part" "0201B103K250NT"
 			(at 148.59 148.59 0)
 			(effects
@@
 			)
 		)
-		(property "JLCPCB Part #" "C338031"
+		(property "JLCPCB Part #" "C285010"
 			(at 127 148.59 0)
 			(effects
@@
 			)
 		)
-		(property "Part" "C0603X5R1A103KT00NN"
+		(property "Part" "0201B103K250NT"
 			(at 127 148.59 0)
 			(effects
@@
 			)
 		)
-		(property "JLCPCB Part #" "C338031"
+		(property "JLCPCB Part #" "C285010"
 			(at 212.09 147.32 0)
 			(effects
@@
 			)
 		)
-		(property "Part" "C0603X5R1A103KT00NN"
+		(property "Part" "0201B103K250NT"
 			(at 212.09 147.32 0)
 			(effects
@@
 			)
 		)
-		(property "JLCPCB Part #" "C338031"
+		(property "JLCPCB Part #" "C285010"
 			(at 316.23 149.86 0)
 			(effects
@@
 			)
 		)
-		(property "Part" "C0603X5R1A103KT00NN"
+		(property "Part" "0201B103K250NT"
 			(at 316.23 149.86 0)
 			(effects
@@
 			)
 		)
-		(property "JLCPCB Part #" "C338031"
+		(property "JLCPCB Part #" "C285010"
 			(at 233.68 147.32 0)
 			(effects
@@
 			)
 		)
-		(property "Part" "C0603X5R1A103KT00NN"
+		(property "Part" "0201B103K250NT"
 			(at 233.68 147.32 0)
 			(effects
@@
 			)
 		)
-		(property "JLCPCB Part #" "C338031"
+		(property "JLCPCB Part #" "C285010"
 			(at 306.07 149.86 0)
 			(effects
@@
 			)
 		)
-		(property "Part" "C0603X5R1A103KT00NN"
+		(property "Part" "0201B103K250NT"
 			(at 306.07 149.86 0)
 			(effects
@@
 			)
 		)
-		(property "JLCPCB Part #" "C338031"
+		(property "JLCPCB Part #" "C285010"
 			(at 138.43 148.59 0)
 			(effects
@@
 			)
 		)
-		(property "Part" "C0603X5R1A103KT00NN"
+		(property "Part" "0201B103K250NT"
 			(at 138.43 148.59 0)
 			(effects
@@
 			)
 		)
-		(property "JLCPCB Part #" "C338031"
+		(property "JLCPCB Part #" "C285010"
 			(at 295.91 149.86 0)
 			(effects
@@
 			)
 		)
-		(property "Part" "C0603X5R1A103KT00NN"
+		(property "Part" "0201B103K250NT"
 			(at 295.91 149.86 0)
 			(effects
@@
 			)
 		)
-		(property "JLCPCB Part #" "C338031"
+		(property "JLCPCB Part #" "C285010"
 			(at 359.41 147.32 0)
 			(effects
@@
 			)
 		)
-		(property "Part" "C0603X5R1A103KT00NN"
+		(property "Part" "0201B103K250NT"
 			(at 359.41 147.32 0)
 			(effects
@@
 			)
 		)
-		(property "JLCPCB Part #" "C338031"
+		(property "JLCPCB Part #" "C285010"
 			(at 223.52 147.32 0)
 			(effects
@@
 			)
 		)
-		(property "Part" "C0603X5R1A103KT00NN"
+		(property "Part" "0201B103K250NT"
 			(at 223.52 147.32 0)
 			(effects
@@
 			)
 		)
-		(property "JLCPCB Part #" "C338031"
+		(property "JLCPCB Part #" "C285010"
 			(at 400.05 147.32 0)
 			(effects
@@
 			)
 		)
-		(property "Part" "C0603X5R1A103KT00NN"
+		(property "Part" "0201B103K250NT"
 			(at 400.05 147.32 0)
 			(effects
@@
 			)
 		)
-		(property "JLCPCB Part #" "C338031"
+		(property "JLCPCB Part #" "C285010"
 			(at 254 147.32 0)
 			(effects
@@
 			)
 		)
-		(property "Part" "C0603X5R1A103KT00NN"
+		(property "Part" "0201B103K250NT"
 			(at 254 147.32 0)
 			(effects

Commit message: JLCPCB id's
Parts:
- C238, C240, C242, C244, C247, C256, C259, C261, C265, C270, C274, C275, C278, C279, C281, C285, C287, C289, C291: Part (none) -> CL03A224MQ3NNNC
Changed lines of the file:
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@@
 			)
 		)
-		(property "Part" ""
+		(property "Part" "CL03A224MQ3NNNC"
 			(at 222.25 135.89 0)
 			(effects
@@
 			)
 		)
-		(property "Part" ""
+		(property "Part" "CL03A224MQ3NNNC"
 			(at 232.41 135.89 0)
 			(effects
@@
 			)
 		)
-		(property "Part" ""
+		(property "Part" "CL03A224MQ3NNNC"
 			(at 294.64 135.89 0)
 			(effects
@@
 			)
 		)
-		(property "Part" ""
+		(property "Part" "CL03A224MQ3NNNC"
 			(at 389.89 135.89 0)
 			(effects
@@
 			)
 		)
-		(property "Part" ""
+		(property "Part" "CL03A224MQ3NNNC"
 			(at 242.57 135.89 0)
 			(effects
@@
 			)
 		)
-		(property "Part" ""
+		(property "Part" "CL03A224MQ3NNNC"
 			(at 147.32 135.89 0)
 			(effects
@@
 			)
 		)
-		(property "Part" ""
+		(property "Part" "CL03A224MQ3NNNC"
 			(at 300.99 114.3 0)
 			(effects
@@
 			)
 		)
-		(property "Part" ""
+		(property "Part" "CL03A224MQ3NNNC"
 			(at 252.73 135.89 0)
 			(effects
@@
 			)
 		)
-		(property "Part" ""
+		(property "Part" "CL03A224MQ3NNNC"
 			(at 304.8 135.89 0)
 			(effects
@@
 			)
 		)
-		(property "Part" ""
+		(property "Part" "CL03A224MQ3NNNC"
 			(at 400.05 135.89 0)
 			(effects
@@
 			)
 		)
-		(property "Part" ""
+		(property "Part" "CL03A224MQ3NNNC"
 			(at 142.24 114.3 0)
 			(effects
@@
 			)
 		)
-		(property "Part" ""
+		(property "Part" "CL03A224MQ3NNNC"
 			(at 379.73 135.89 0)
 			(effects
@@
 			)
 		)
-		(property "Part" ""
+		(property "Part" "CL03A224MQ3NNNC"
 			(at 167.64 135.89 0)
 			(effects
@@
 			)
 		)
-		(property "Part" ""
+		(property "Part" "CL03A224MQ3NNNC"
 			(at 153.67 114.3 0)
 			(effects
@@
 			)
 		)
-		(property "Part" ""
+		(property "Part" "CL03A224MQ3NNNC"
 			(at 314.96 135.89 0)
 			(effects
@@
 			)
 		)
-		(property "Part" ""
+		(property "Part" "CL03A224MQ3NNNC"
 			(at 289.56 114.3 0)
 			(effects
@@
 			)
 		)
-		(property "Part" ""
+		(property "Part" "CL03A224MQ3NNNC"
 			(at 369.57 135.89 0)
 			(effects
@@
 			)
 		)
-		(property "Part" ""
+		(property "Part" "CL03A224MQ3NNNC"
 			(at 157.48 135.89 0)
 			(effects
@@
 			)
 		)
-		(property "Part" ""
+		(property "Part" "CL03A224MQ3NNNC"
 			(at 284.48 135.89 0)
 			(effects
