File: psddr3.kicad_sch (KiCad schematic)
At the start: 103 parts, among them U21 XC7Z030_FBG676, U27 MT41K256M16TW-107:P, U28 TPS51200DRC, U29 MT41K256M16TW-107:P

Commit message: schema: DDR termination resistors to 100Ohm
Parts:
- R200, R201: value 80.6 1% -> 100 1%; JLCPCB Part # C25134 -> C25076; Part 0402WGF806JTCE -> 0402WGF1000TCE
- R226: JLCPCB Part # C153111 -> C25076; Part RM04FTN1000 -> 0402WGF1000TCE
Changed lines of the file:
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@@
 			)
 		)
-		(property "Value" "80.6 1%"
+		(property "Value" "100 1%"
 			(at 17.145 118.11 0)
 			(effects
@@
 			)
 		)
-		(property "JLCPCB Part #" "C25134"
+		(property "JLCPCB Part #" "C25076"
 			(at 15.24 116.84 0)
 			(effects
@@
 			)
 		)
-		(property "Part" "0402WGF806JTCE"
+		(property "Part" "0402WGF1000TCE"
 			(at 15.24 116.84 0)
 			(effects
@@
 			)
 		)
-		(property "JLCPCB Part #" "C153111"
+		(property "JLCPCB Part #" "C25076"
 			(at 67.31 250.19 0)
 			(effects
@@
 			)
 		)
-		(property "Part" "RM04FTN1000"
+		(property "Part" "0402WGF1000TCE"
 			(at 67.31 250.19 0)
 			(effects
@@
 			)
 		)
-		(property "Value" "80.6 1%"
+		(property "Value" "100 1%"
 			(at 17.145 107.95 0)
 			(effects
@@
 			)
 		)
-		(property "JLCPCB Part #" "C25134"
+		(property "JLCPCB Part #" "C25076"
 			(at 15.24 106.68 0)
 			(effects
@@
 			)
 		)
-		(property "Part" "0402WGF806JTCE"
+		(property "Part" "0402WGF1000TCE"
 			(at 15.24 106.68 0)
 			(effects
