File: psddr3.kicad_sch (KiCad schematic)
At the start: 103 parts, among them U21 XC7Z030_FBG676, U27 MT41K256M16TW-107:P, U28 TPS51200DRC, U29 MT41K256M16TW-107:P

Commit message: JLCPCB ID attribute updates
These 'JLCPCB Part #' updates reflect the JLCPCB assembly order # SMT026073061946-2250854A
Parts:
- R227: JLCPCB Part # C25900 -> C105871; Part 0402WGF4701TCE -> RC0402FR-074K7L
Changed lines of the file:
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@@
 			)
 		)
-		(property "JLCPCB Part #" "C25900"
+		(property "JLCPCB Part #" "C105871"
 			(at 67.31 261.62 0)
 			(effects
@@
 			)
 		)
-		(property "Part" "0402WGF4701TCE"
+		(property "Part" "RC0402FR-074K7L"
 			(at 67.31 261.62 0)
 			(effects
