File: soc_power.kicad_sch (KiCad schematic)
At the start: 145 parts, among them IC1 NL17SZ17XV5T2G, IC2 TLV74325PDBVR, Q5 FDS9926A, Q6 BSS138, Q7 BSS138, Q8 BSS138, U2 ADP5052ACPZ-R7, U3 LD1117S12TR, U4 AZ1117H-ADJTRG1, U5 SN74LXC1T45DBVR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

Commit message: jlcpcb id's update
Parts:
- R48, R52: JLCPCB Part # C705933 -> C22772; Part RT0603DRD0710K2L -> 0603WAF1022T5E
Changed lines of the file:
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@@
 			)
 		)
-		(property "JLCPCB Part #" "C705933"
+		(property "JLCPCB Part #" "C22772"
 			(at 175.26 22.86 0)
 			(effects
@@
 			)
 		)
-		(property "Part" "RT0603DRD0710K2L"
+		(property "Part" "0603WAF1022T5E"
 			(at 175.26 22.86 90)
 			(effects
@@
 			)
 		)
-		(property "JLCPCB Part #" "C705933"
+		(property "JLCPCB Part #" "C22772"
 			(at 164.465 105.41 0)
 			(effects
@@
 			)
 		)
-		(property "Part" "RT0603DRD0710K2L"
+		(property "Part" "0603WAF1022T5E"
 			(at 164.465 105.41 90)
 			(effects

Commit message: JLCPCB id's
Parts:
- L1, L2, L3: Part 0412CDMCCDS-3R3MC -> 0412CDMCCDS-3R3MC
Changed lines of the file:
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@@
 			)
 		)
-		(property "Part" "    0412CDMCCDS-3R3MC"
+		(property "Part" "0412CDMCCDS-3R3MC"
 			(at 173.355 76.2 0)
 			(effects
@@
 			)
 		)
-		(property "Part" "    0412CDMCCDS-3R3MC"
+		(property "Part" "0412CDMCCDS-3R3MC"
 			(at 173.355 99.06 0)
 			(effects
@@
 			)
 		)
-		(property "Part" "    0412CDMCCDS-3R3MC"
+		(property "Part" "0412CDMCCDS-3R3MC"
 			(at 201.295 33.02 0)
 			(effects

Commit message: more powerful inductors for SOC SMPS
Parts:
- L1, L2, L3: footprint pretty:0412CDMCCDS -> pretty:SRYH.0530.YF3R3MT00; JLCPCB Part # C2453260 -> C5122863; Part 0412CDMCCDS-3R3MC -> SRYH.0530.YF3R3MT00
Changed lines of the file:
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@@
 			)
 		)
-		(property "Footprint" "pretty:0412CDMCCDS"
+		(property "Footprint" "pretty:SRYH.0530.YF3R3MT00"
 			(at 173.355 76.2 0)
 			(effects
@@
 			)
 		)
-		(property "Description" ""
+		(property "Description" "3.3uH 4.5A 45mΩ 7A ±20% SMD,5.6x5.3mm Power Inductors ROHS"
 			(at 173.355 76.2 0)
 			(effects
@@
 			)
 		)
-		(property "JLCPCB Part #" "C2453260"
+		(property "JLCPCB Part #" "C5122863"
 			(at 173.355 76.2 0)
 			(effects
@@
 			)
 		)
-		(property "Part" "0412CDMCCDS-3R3MC"
+		(property "Part" "SRYH.0530.YF3R3MT00"
 			(at 173.355 76.2 0)
 			(effects
@@
 			)
 		)
-		(property "Footprint" "pretty:0412CDMCCDS"
+		(property "Footprint" "pretty:SRYH.0530.YF3R3MT00"
 			(at 173.355 99.06 0)
 			(effects
@@
 			)
 		)
-		(property "Description" ""
+		(property "Description" "3.3uH 4.5A 45mΩ 7A ±20% SMD,5.6x5.3mm Power Inductors ROHS"
 			(at 173.355 99.06 0)
 			(effects
@@
 			)
 		)
-		(property "JLCPCB Part #" "C2453260"
+		(property "JLCPCB Part #" "C5122863"
 			(at 173.355 99.06 0)
 			(effects
@@
 			)
 		)
-		(property "Part" "0412CDMCCDS-3R3MC"
+		(property "Part" "SRYH.0530.YF3R3MT00"
 			(at 173.355 99.06 0)
 			(effects
@@
 			)
 		)
-		(property "Footprint" "pretty:0412CDMCCDS"
+		(property "Footprint" "pretty:SRYH.0530.YF3R3MT00"
 			(at 201.295 33.02 0)
 			(effects
@@
 			)
 		)
-		(property "Description" ""
+		(property "Description" "3.3uH 4.5A 45mΩ 7A ±20% SMD,5.6x5.3mm Power Inductors ROHS"
 			(at 201.295 33.02 0)
 			(effects
@@
 			)
 		)
-		(property "JLCPCB Part #" "C2453260"
+		(property "JLCPCB Part #" "C5122863"
 			(at 201.295 33.02 0)
 			(effects
@@
 			)
 		)
-		(property "Part" "0412CDMCCDS-3R3MC"
+		(property "Part" "SRYH.0530.YF3R3MT00"
 			(at 201.295 33.02 0)
 			(effects
