File: soc_power.kicad_sch (KiCad schematic)
At the start: 145 parts, among them IC1 NL17SZ17XV5T2G, IC2 TLV74325PDBVR, Q5 FDS9926A, Q6 BSS138, Q7 BSS138, Q8 BSS138, U2 ADP5052ACPZ-R7, U3 LD1117S12TR, U4 AZ1117H-ADJTRG1, U5 SN74LXC1T45DBVR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

Commit message: schema: external clock input redone
Parts:
- L1, L2, L3: Alt (none) -> ASPI-0520LR-3R3M-T2
Changed lines of the file:
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@@
 			)
 		)
+		(property "Alt" "ASPI-0520LR-3R3M-T2"
+			(at 173.355 76.2 90)
+			(effects
+				(font
+					(size 1.27 1.27)
+				)
+				(hide yes)
+			)
+		)
 		(pin "2"
 		)
@@
 			)
 		)
+		(property "Alt" "ASPI-0520LR-3R3M-T2"
+			(at 173.355 99.06 90)
+			(effects
+				(font
+					(size 1.27 1.27)
+				)
+				(hide yes)
+			)
+		)
 		(pin "2"
 		)
@@
 			(at 201.295 33.02 90)
 			(effects
+				(font
+					(size 1.27 1.27)
+				)
+				(hide yes)
+			)
+		)
+		(property "Alt" "ASPI-0520LR-3R3M-T2"
+			(at 201.295 33.02 90)
+			(effects

Commit message: schema: AC term of SOC primary clock
AC term of primary 33.333 clock
ERRATA updates
Parts:
- L4: JLCPCB Part # C135227 -> C53281631; Part SMNR3010-1R5MT -> FTC303015D1R5MBCA
Changed lines of the file:
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@@
 			)
 		)
-		(property "JLCPCB Part #" "C135227"
+		(property "JLCPCB Part #" "C53281631"
 			(at 201.295 57.15 90)
 			(effects
@@
 			)
 		)
-		(property "Part" "SMNR3010-1R5MT"
+		(property "Part" "FTC303015D1R5MBCA"
 			(at 201.295 57.15 90)
 			(effects

Commit message: schema: force PMIC to PWM mode - place R45
Parts:
- R44: now not fitted
- R45: now fitted
Changed lines of the file:
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@@
 		(in_bom yes)
 		(on_board yes)
-		(dnp yes)
+		(dnp no)
 		(fields_autoplaced yes)
 		(property "Reference" "R45"
@@
 		(in_bom yes)
 		(on_board yes)
-		(dnp no)
+		(dnp yes)
 		(fields_autoplaced yes)
 		(property "Reference" "R44"

Commit message: schema: extra leds from the psu were removed
Parts:
- removed D13, D15: LED, LED_SMD:LED_0805_2012Metric, symbol Device:LED
- removed R64, R71: 330, Resistor_SMD:R_0402_1005Metric, symbol Device:R_Small

Commit message: schema: soc core power 1V0 is capped at 6.4A with R51 of 22k
Parts:
- R51: value 47k -> 22k; JLCPCB Part # C5139555 -> C31850; Part (none) -> 0603WAF2202T5E
Other:
- note added: "0.2A"
- note added: "2.5A R50 = 47K unsolder R50 to get 4.4A"
- note added: "6.44A MAX R51 = 22k"
- note removed: "0.6A -2A MAX"
- note removed: "2.1A"
- note removed: "2.5A"
Changed lines of the file:
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@@
 		)
 	)
-	(text "0.6A -2A MAX"
-		(exclude_from_sim no)
-		(at 242.824 96.266 0)
-		(effects
-			(font
-				(size 1.27 1.27)
-			)
-			(justify left bottom)
-		)
-	)
 	(text "PMIC_EN2\nstarts 1V0\n(first pwr bus)"
 		(exclude_from_sim no)
@@
 		)
 	)
-	(text "2.5A"
+	(text "2.5A\nR50 = 47K\nunsolder R50 to get 4.4A"
 		(exclude_from_sim no)
-		(at 268.478 23.622 0)
+		(at 268.732 35.052 0)
 		(effects
 			(font
@@
 		)
 	)
+	(text "0.2A"
+		(exclude_from_sim no)
+		(at 211.836 112.014 0)
+		(effects
+			(font
+				(size 1.27 1.27)
+			)
+			(justify left bottom)
+		)
+	)
 	(text "1.2A"
 		(exclude_from_sim no)
@@
 		)
 	)
+	(text "1.2A"
+		(exclude_from_sim no)
+		(at 242.57 98.298 0)
+		(effects
+			(font
+				(size 1.27 1.27)
+			)
+			(justify left bottom)
+		)
+	)
 	(text "SOC PWR +3V3_SYS is started (last in seq) [OUT] +1V8 signal\n"
 		(exclude_from_sim no)
@@
 		)
 	)
-	(text "2.1A"
+	(text "6.44A MAX\nR51 = 22k"
 		(exclude_from_sim no)
-		(at 313.944 44.45 0)
+		(at 314.96 45.466 0)
 		(effects
 			(font
@@
 			)
 		)
-		(property "Value" "47k"
+		(property "Value" "22k"
 			(at 176.53 50.165 0)
 			(effects
@@
 			)
 		)
-		(property "Description" ""
+		(property "Description" "-55℃~+155℃ 100mW 22kΩ 75V Thick Film Resistor ±1% ±100ppm/℃ 0603 Chip Resistor - Surface Mount ROHS"
 			(at 173.99 48.895 0)
 			(effects
@@
 			)
 		)
-		(property "JLCPCB Part #" "C5139555"
+		(property "JLCPCB Part #" "C31850"
 			(at 173.99 48.895 0)
 			(effects
@@
 			(at 173.99 48.895 0)
 			(effects
+				(font
+					(size 1.27 1.27)
+				)
+				(hide yes)
+			)
+		)
+		(property "Part" "0603WAF2202T5E"
+			(at 173.99 48.895 0)
+			(effects
