File: soc_power.kicad_sch (KiCad schematic)
At the start: 141 parts, among them IC1 NL17SZ17XV5T2G, IC2 TLV74325PDBVR, Q5 FDS9926A, Q6 BSS138, Q7 BSS138, Q8 BSS138, U2 ADP5052ACPZ-R7, U3 LD1117S12TR, U4 AZ1117H-ADJTRG1, U5 SN74LXC1T45DBVR, U52 INA219AxDCN, U53 INA219AxDCN, U54 INA219AxDCN, U6 TPS25940AQRVCRQ1

Commit message: bom: substitute out-of-stock passives, sync descriptions to JLCPCB IDs
Every substitution keeps its existing footprint, so no PCB rework is
implied. Stock figures verified against live LCSC, not the parts-library
snapshot (which was stale on four parts).

  C11-C13  C188358 -> C178366   82uF/35V -> 180uF/25V OS-CON SVPF (was OOS)
  R54      C138285 -> C2933137  12.7k 0603 (was OOS)
  31x tant C1954274 -> C7214    22uF 16V -> 25V; ~16 -> ~2580 boards of
                                stock, and fixes the +12VEXT derating on
                                C430/C431 (75% -> 48% of rating)
  20x cap  C513774 -> C13585    10uF 1206, JLC Basic part
  C76,C77  C2918589 -> C541338  4.3pF +-0.1pF, 32.768kHz load caps for Y2
  R286     C705904 -> C2930124  649R, HX2VL RREF
  R45      C2936632 -> C17477   consolidated onto an existing BOM line
  C328     C2170363 -> C368809  consolidated; was outside the JLC library
  R172     C705658 -> C705678   consolidated; was outside the JLC library

Fix eight capacitors labelled 10nFx50V that carried a 10uF part number:
C31 C32 C302 C307 C309 C347 C360 C368 -> value corrected to 10uFx50V.
All sit on power rails or LDO inputs where 10uF is the intent.

Restore C302's Footprint, which had been corrupted to "c9" (not a valid
library reference; would have failed the next PCB update).

Regenerate Description on all 822 R/C from live LCSC parametric data so
each matches its JLCPCB Part #.

Value fields keep the project convention: the voltage suffix is the design
minimum, not the fitted part's rating, so the tantalum stayed 22uFx16V.
C11-C13 did change 82uF -> 180uF because the capacitance itself changed.

Also carries work in progress from this session: H35 mounting hole,
R50/R137/R285 moved to 0402 (C25792), R30 220R -> 330R (C5154013),
C24 -> C1618.

NASR.net and NASR.kicad_pcb still predate these schematic edits; they need
a netlist re-export and Update PCB from Schematic.

Co-Authored-By: Claude Opus 5 (1M context) <noreply@anthropic.c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
Parts:
- C21, C22, C27, C28, C34, C36: JLCPCB Part # C1954274 -> C7214; Part TR3C226K016C0350 -> TAJC226K025RNJ
- C24: JLCPCB Part # C470850 -> C1618; Part GRM188R71H392KA01D -> 0603B392K500NT
- C31, C32: value 10nFx50V -> 10uFx50V; JLCPCB Part # C513774 -> C13585; Part (none) -> CL31A106KBHNNNE
- R45: JLCPCB Part # C2936632 -> C17477; Part (none) -> 0805W8F0000T5E
- R50: footprint Resistor_SMD:R_0603_1608Metric -> Resistor_SMD:R_0402_1005Metric; JLCPCB Part # C5139555 -> C25792; Part (none) -> 0402WGF4702TCE
- R54: JLCPCB Part # C138285 -> C2933137; Part AC0603FR-0712K7L -> FRC0603F1272TS
