File: soc_power.kicad_sch (KiCad schematic)
At the start: 141 parts, among them IC1 NL17SZ17XV5T2G, IC2 TLV74325PDBVR, Q5 FDS9926A, Q6 BSS138, Q7 BSS138, Q8 BSS138, U2 ADP5052ACPZ-R7, U3 LD1117S12TR, U4 AZ1117H-ADJTRG1, U5 SN74LXC1T45DBVR, U52 INA219AxDCN, U53 INA219AxDCN, U54 INA219AxDCN, U6 TPS25940AQRVCRQ1

Commit message: JLCPCB ID attribute updates
These 'JLCPCB Part #' updates reflect the JLCPCB assembly order # SMT026073061946-2250854A
Parts:
- R321, R322, R323, R324, R325, R326: JLCPCB Part # C102766 -> C22369459; Part RTT0210R0FTH -> RCA0210RFLF
- R36, R40, R59, R75: JLCPCB Part # C25900 -> C105871; Part 0402WGF4701TCE -> RC0402FR-074K7L
- R47: JLCPCB Part # C245945 -> C2998119; Part RC0603FR-0728K7L -> FRC0603F2872TS
Changed lines of the file:
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@@
 			)
 		)
-		(property "JLCPCB Part #" "C25900"
+		(property "JLCPCB Part #" "C105871"
 			(at 73.66 69.85 0)
 			(effects
@@
 			)
 		)
-		(property "Part" "0402WGF4701TCE"
+		(property "Part" "RC0402FR-074K7L"
 			(at 73.66 69.85 0)
 			(effects
@@
 			)
 		)
-		(property "Description" "-55℃~+155℃ 10Ω 50V 62.5mW Thick Film Resistor ±1% ±100ppm/℃ 0402 Chip Resistor - Surface Mount ROHS"
+		(property "Description" "-55℃~+155℃ 10Ω 50V 62.5mW Thick Film Resistor ±1% ±400ppm/℃ 0402 Chip Resistor - Surface Mount ROHS"
 			(at 238.76 207.01 0)
 			(effects
@@
 			)
 		)
-		(property "JLCPCB Part #" "C102766"
+		(property "JLCPCB Part #" "C22369459"
 			(at 238.76 207.01 0)
 			(effects
@@
 			)
 		)
-		(property "Part" "RTT0210R0FTH"
+		(property "Part" "RCA0210RFLF"
 			(at 238.76 207.01 0)
 			(effects
@@
 			)
 		)
-		(property "Description" "-55℃~+155℃ 10Ω 50V 62.5mW Thick Film Resistor ±1% ±100ppm/℃ 0402 Chip Resistor - Surface Mount ROHS"
+		(property "Description" "-55℃~+155℃ 10Ω 50V 62.5mW Thick Film Resistor ±1% ±400ppm/℃ 0402 Chip Resistor - Surface Mount ROHS"
 			(at 238.76 157.48 0)
 			(effects
@@
 			)
 		)
-		(property "JLCPCB Part #" "C102766"
+		(property "JLCPCB Part #" "C22369459"
 			(at 238.76 157.48 0)
 			(effects
@@
 			)
 		)
-		(property "Part" "RTT0210R0FTH"
+		(property "Part" "RCA0210RFLF"
 			(at 238.76 157.48 0)
 			(effects
@@
 			)
 		)
-		(property "JLCPCB Part #" "C25900"
+		(property "JLCPCB Part #" "C105871"
 			(at 38.1 35.56 0)
 			(effects
@@
 			)
 		)
-		(property "Part" "0402WGF4701TCE"
+		(property "Part" "RC0402FR-074K7L"
 			(at 38.1 35.56 0)
 			(effects
@@
 			)
 		)
-		(property "Description" "-55℃~+155℃ 10Ω 50V 62.5mW Thick Film Resistor ±1% ±100ppm/℃ 0402 Chip Resistor - Surface Mount ROHS"
+		(property "Description" "-55℃~+155℃ 10Ω 50V 62.5mW Thick Film Resistor ±1% ±400ppm/℃ 0402 Chip Resistor - Surface Mount ROHS"
 			(at 238.76 162.56 0)
 			(effects
@@
 			)
 		)
-		(property "JLCPCB Part #" "C102766"
+		(property "JLCPCB Part #" "C22369459"
 			(at 238.76 162.56 0)
 			(effects
@@
 			)
 		)
-		(property "Part" "RTT0210R0FTH"
+		(property "Part" "RCA0210RFLF"
 			(at 238.76 162.56 0)
 			(effects
@@
 			)
 		)
-		(property "Description" "-55℃~+155℃ 10Ω 50V 62.5mW Thick Film Resistor ±1% ±100ppm/℃ 0402 Chip Resistor - Surface Mount ROHS"
+		(property "Description" "-55℃~+155℃ 10Ω 50V 62.5mW Thick Film Resistor ±1% ±400ppm/℃ 0402 Chip Resistor - Surface Mount ROHS"
 			(at 238.76 252.73 0)
 			(effects
@@
 			)
 		)
-		(property "JLCPCB Part #" "C102766"
+		(property "JLCPCB Part #" "C22369459"
 			(at 238.76 252.73 0)
 			(effects
@@
 			)
 		)
-		(property "Part" "RTT0210R0FTH"
+		(property "Part" "RCA0210RFLF"
 			(at 238.76 252.73 0)
 			(effects
@@
 			)
 		)
-		(property "Description" "-55℃~+155℃ 28.7kΩ 75V 100mW Thick Film Resistor ±1% ±100ppm/℃ 0603 Chip Resistor - Surface Mount ROHS"
+		(property "Description" "-55℃~+155℃ 100mW 28.7kΩ 75V Thick Film Resistor ±1% ±100ppm/℃ 0603 Chip Resistor - Surface Mount ROHS"
 			(at 164.465 82.55 0)
 			(effects
@@
 			)
 		)
-		(property "JLCPCB Part #" "C245945"
+		(property "JLCPCB Part #" "C2998119"
 			(at 164.465 82.55 0)
 			(effects
@@
 			)
 		)
-		(property "Part" "RC0603FR-0728K7L"
+		(property "Part" "FRC0603F2872TS"
 			(at 164.465 82.55 90)
 			(effects
@@
 			)
 		)
-		(property "Description" "-55℃~+155℃ 10Ω 50V 62.5mW Thick Film Resistor ±1% ±100ppm/℃ 0402 Chip Resistor - Surface Mount ROHS"
+		(property "Description" "-55℃~+155℃ 10Ω 50V 62.5mW Thick Film Resistor ±1% ±400ppm/℃ 0402 Chip Resistor - Surface Mount ROHS"
 			(at 238.76 247.65 0)
 			(effects
@@
 			)
 		)
-		(property "JLCPCB Part #" "C102766"
+		(property "JLCPCB Part #" "C22369459"
 			(at 238.76 247.65 0)
 			(effects
@@
 			)
 		)
-		(property "Part" "RTT0210R0FTH"
+		(property "Part" "RCA0210RFLF"
 			(at 238.76 247.65 0)
 			(effects
@@
 			)
 		)
-		(property "JLCPCB Part #" "C25900"
+		(property "JLCPCB Part #" "C105871"
 			(at 323.85 113.03 0)
 			(effects
@@
 			)
 		)
-		(property "Part" "0402WGF4701TCE"
+		(property "Part" "RC0402FR-074K7L"
 			(at 323.85 113.03 0)
 			(effects
@@
 			)
 		)
-		(property "Description" "-55℃~+155℃ 10Ω 50V 62.5mW Thick Film Resistor ±1% ±100ppm/℃ 0402 Chip Resistor - Surface Mount ROHS"
+		(property "Description" "-55℃~+155℃ 10Ω 50V 62.5mW Thick Film Resistor ±1% ±400ppm/℃ 0402 Chip Resistor - Surface Mount ROHS"
 			(at 238.76 201.93 0)
 			(effects
@@
 			)
 		)
-		(property "JLCPCB Part #" "C102766"
+		(property "JLCPCB Part #" "C22369459"
 			(at 238.76 201.93 0)
 			(effects
@@
 			)
 		)
-		(property "Part" "RTT0210R0FTH"
+		(property "Part" "RCA0210RFLF"
 			(at 238.76 201.93 0)
 			(effects
@@
 			)
 		)
-		(property "JLCPCB Part #" "C25900"
+		(property "JLCPCB Part #" "C105871"
 			(at 200.66 187.96 0)
 			(effects
@@
 			)
 		)
-		(property "Part" "0402WGF4701TCE"
+		(property "Part" "RC0402FR-074K7L"
 			(at 200.66 187.96 0)
 			(effects
