File: NASR.kicad_sch (KiCad schematic)
At the start: 21 parts

Commit message: bom: substitute out-of-stock passives, sync descriptions to JLCPCB IDs
Every substitution keeps its existing footprint, so no PCB rework is
implied. Stock figures verified against live LCSC, not the parts-library
snapshot (which was stale on four parts).

  C11-C13  C188358 -> C178366   82uF/35V -> 180uF/25V OS-CON SVPF (was OOS)
  R54      C138285 -> C2933137  12.7k 0603 (was OOS)
  31x tant C1954274 -> C7214    22uF 16V -> 25V; ~16 -> ~2580 boards of
                                stock, and fixes the +12VEXT derating on
                                C430/C431 (75% -> 48% of rating)
  20x cap  C513774 -> C13585    10uF 1206, JLC Basic part
  C76,C77  C2918589 -> C541338  4.3pF +-0.1pF, 32.768kHz load caps for Y2
  R286     C705904 -> C2930124  649R, HX2VL RREF
  R45      C2936632 -> C17477   consolidated onto an existing BOM line
  C328     C2170363 -> C368809  consolidated; was outside the JLC library
  R172     C705658 -> C705678   consolidated; was outside the JLC library

Fix eight capacitors labelled 10nFx50V that carried a 10uF part number:
C31 C32 C302 C307 C309 C347 C360 C368 -> value corrected to 10uFx50V.
All sit on power rails or LDO inputs where 10uF is the intent.

Restore C302's Footprint, which had been corrupted to "c9" (not a valid
library reference; would have failed the next PCB update).

Regenerate Description on all 822 R/C from live LCSC parametric data so
each matches its JLCPCB Part #.

Value fields keep the project convention: the voltage suffix is the design
minimum, not the fitted part's rating, so the tantalum stayed 22uFx16V.
C11-C13 did change 82uF -> 180uF because the capacitance itself changed.

Also carries work in progress from this session: H35 mounting hole,
R50/R137/R285 moved to 0402 (C25792), R30 220R -> 330R (C5154013),
C24 -> C1618.

NASR.net and NASR.kicad_pcb still predate these schematic edits; they need
a netlist re-export and Update PCB from Schematic.

Co-Authored-By: Claude Opus 5 (1M context) <noreply@anthropic.c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
Parts:
- added H34, H35: MH4_M3, MountingHole:MountingHole_3.2mm_M3_Pad_Via, symbol Mechanical:MountingHole_Pad
Changed lines of the file:
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@@
+	)
+	(symbol
+		(lib_id "Mechanical:MountingHole_Pad")
+		(at 146.05 260.35 0)
+		(unit 1)
+		(exclude_from_sim yes)
+		(in_bom no)
+		(on_board yes)
+		(dnp no)
+		(fields_autoplaced yes)
+		(property "Reference" "H35"
+			(at 148.59 257.8099 0)
+			(effects
+				(font
+					(size 1.27 1.27)
+				)
+				(justify left)
+			)
+		)
+		(property "Value" "MH4_M3"
+			(at 148.59 260.3499 0)
+			(effects
+				(font
+					(size 1.27 1.27)
+				)
+				(justify left)
+			)
+		)
+		(property "Footprint" "MountingHole:MountingHole_3.2mm_M3_Pad_Via"
+			(at 146.05 260.35 0)
+			(effects
+				(font
+					(size 1.27 1.27)
+				)
+				(hide yes)
+			)
+		)
+		(property "Datasheet" "~"
+			(at 146.05 260.35 0)
+			(effects
+				(font
+					(size 1.27 1.27)
+				)
+				(hide yes)
+			)
+		)
+		(property "Description" "Mounting Hole with connection"
+			(at 146.05 260.35 0)
+			(effects
+				(font
+					(size 1.27 1.27)
+				)
+				(hide yes)
+			)
+		)
+		(property "Mouser " ""
+			(at 146.05 260.35 0)
+			(effects
+				(font
+					(size 1.27 1.27)
+				)
+				(hide yes)
+			)
+		)
+		(pin "1"
+		)
+		(instances
+			(project "NASR"
+				(path "/9a13c8f9-b8a2-41aa-b5bd-813f44236e01"
+					(reference "H35")
+					(unit 1)
+				)
+			)
+		)
 	)
 	(symbol
@@
 			)
 		)
-		(property "Description" ""
+		(property "Description" "-55℃~+155℃ 0Ω 200V 500mW Thick Film Resistor ±5% 1210 Chip Resistor - Surface Mount ROHS"
 			(at 21.59 271.78 0)
 			(effects
@@
 					(unit 1)
 				)
+			)
+		)
+	)
+	(symbol
+		(lib_id "Mechanical:MountingHole_Pad")
+		(at 125.73 260.35 0)
+		(unit 1)
+		(exclude_from_sim yes)
+		(in_bom no)
+		(on_board yes)
+		(dnp no)
+		(fields_autoplaced yes)
+		(property "Reference" "H34"
+			(at 128.27 257.8099 0)
+			(effects
+				(font
+					(size 1.27 1.27)
+				)
+				(justify left)
+			)
+		)
+		(property "Value" "MH4_M3"
+			(at 128.27 260.3499 0)
+			(effects
+				(font
+					(size 1.27 1.27)
+				)
+				(justify left)
+			)
+		)
+		(property "Footprint" "MountingHole:MountingHole_3.2mm_M3_Pad_Via"
+			(at 125.73 260.35 0)
+			(effects
+				(font
+					(size 1.27 1.27)
+				)
+				(hide yes)
+			)
+		)
+		(property "Datasheet" "~"
+			(at 125.73 260.35 0)
+			(effects
+				(font
+					(size 1.27 1.27)
+				)
+				(hide yes)
+			)
+		)
+		(property "Description" "Mounting Hole with connection"
+			(at 125.73 260.35 0)
+			(effects
+				(font
+					(size 1.27 1.27)
+				)
+				(hide yes)
+			)
+		)
+		(property "Mouser " ""
+			(at 125.73 260.35 0)
+			(effects
+				(font
+					(size 1.27 1.27)
+				)
+				(hide yes)
+			)
+		)
+		(pin "1"
+		)
+		(instances
+			(project "NASR"
+				(path "/9a13c8f9-b8a2-41aa-b5bd-813f44236e01"
+					(reference "H34")
+					(unit 1)
+				)
