File: syzygy34.kicad_sch (KiCad schematic)
At the start: 55 parts, among them J30 292161-3, J31 292161-3, J32 SYZYGY_SOCKET-STD, J33 SYZYGY_SOCKET-STD, U21 XC7Z030_FBG676

Commit message: +12VEXT on SYZYGY pin 38 to power up analog circuitry on pods
Parts:
- added C430, C431: 22uFx16V, Capacitor_Tantalum_SMD:CP_EIA-6032-15_Kemet-U, symbol Device:C_Polarized
Connections:
- net GND: now also C430.2, C431.2
- net +12VEXT: now reaches J33.38 (RSVD)
- net +12VEXT: now also J32.38 (RSVD), C430.1, C431.1
- no-connect marks 50 -> 48
