File: eth_ps.kicad_sch (KiCad schematic)
At the start: 41 parts, among them J24 RJ45_RB1-125B8G1A, U32 RTL8211F-CG, Y4 SX5B25.000F1220F30

Commit message: JLCPCB ID attribute updates
These 'JLCPCB Part #' updates reflect the JLCPCB assembly order # SMT026073061946-2250854A
Parts:
- R260, R261, R262, R263, R264, R265, R267, R271, R272, R273, R274, R275, R276: JLCPCB Part # C25900 -> C105871; Part 0402WGF4701TCE -> RC0402FR-074K7L
Changed lines of the file:
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@@
 			)
 		)
-		(property "JLCPCB Part #" "C25900"
+		(property "JLCPCB Part #" "C105871"
 			(at 95.25 72.39 0)
 			(effects
@@
 			)
 		)
-		(property "Part" "0402WGF4701TCE"
+		(property "Part" "RC0402FR-074K7L"
 			(at 95.25 72.39 0)
 			(effects
@@
 			)
 		)
-		(property "JLCPCB Part #" "C25900"
+		(property "JLCPCB Part #" "C105871"
 			(at 82.55 251.46 0)
 			(effects
@@
 			)
 		)
-		(property "Part" "0402WGF4701TCE"
+		(property "Part" "RC0402FR-074K7L"
 			(at 82.55 251.46 0)
 			(effects
@@
 			)
 		)
-		(property "JLCPCB Part #" "C25900"
+		(property "JLCPCB Part #" "C105871"
 			(at 92.71 254 0)
 			(effects
@@
 			)
 		)
-		(property "Part" "0402WGF4701TCE"
+		(property "Part" "RC0402FR-074K7L"
 			(at 92.71 254 0)
 			(effects
@@
 			)
 		)
-		(property "JLCPCB Part #" "C25900"
+		(property "JLCPCB Part #" "C105871"
 			(at 347.98 165.1 0)
 			(effects
@@
 			)
 		)
-		(property "Part" "0402WGF4701TCE"
+		(property "Part" "RC0402FR-074K7L"
 			(at 347.98 165.1 0)
 			(effects
@@
 			)
 		)
-		(property "JLCPCB Part #" "C25900"
+		(property "JLCPCB Part #" "C105871"
 			(at 396.24 165.1 0)
 			(effects
@@
 			)
 		)
-		(property "Part" "0402WGF4701TCE"
+		(property "Part" "RC0402FR-074K7L"
 			(at 396.24 165.1 0)
 			(effects
@@
 			)
 		)
-		(property "JLCPCB Part #" "C25900"
+		(property "JLCPCB Part #" "C105871"
 			(at 347.98 176.53 0)
 			(effects
@@
 			)
 		)
-		(property "Part" "0402WGF4701TCE"
+		(property "Part" "RC0402FR-074K7L"
 			(at 347.98 176.53 0)
 			(effects
@@
 			)
 		)
-		(property "JLCPCB Part #" "C25900"
+		(property "JLCPCB Part #" "C105871"
 			(at 90.17 245.11 0)
 			(effects
@@
 			)
 		)
-		(property "Part" "0402WGF4701TCE"
+		(property "Part" "RC0402FR-074K7L"
 			(at 90.17 245.11 0)
 			(effects
@@
 			)
 		)
-		(property "JLCPCB Part #" "C25900"
+		(property "JLCPCB Part #" "C105871"
 			(at 90.17 240.03 0)
 			(effects
@@
 			)
 		)
-		(property "Part" "0402WGF4701TCE"
+		(property "Part" "RC0402FR-074K7L"
 			(at 90.17 240.03 0)
 			(effects
@@
 			)
 		)
-		(property "JLCPCB Part #" "C25900"
+		(property "JLCPCB Part #" "C105871"
 			(at 77.47 237.49 0)
 			(effects
@@
 			)
 		)
-		(property "Part" "0402WGF4701TCE"
+		(property "Part" "RC0402FR-074K7L"
 			(at 77.47 237.49 0)
 			(effects
@@
 			)
 		)
-		(property "JLCPCB Part #" "C25900"
+		(property "JLCPCB Part #" "C105871"
 			(at 77.47 242.57 0)
 			(effects
@@
 			)
 		)
-		(property "Part" "0402WGF4701TCE"
+		(property "Part" "RC0402FR-074K7L"
 			(at 77.47 242.57 0)
 			(effects
@@
 			)
 		)
-		(property "JLCPCB Part #" "C25900"
+		(property "JLCPCB Part #" "C105871"
 			(at 396.24 176.53 0)
 			(effects
@@
 			)
 		)
-		(property "Part" "0402WGF4701TCE"
+		(property "Part" "RC0402FR-074K7L"
 			(at 396.24 176.53 0)
 			(effects
@@
 			)
 		)
-		(property "JLCPCB Part #" "C25900"
+		(property "JLCPCB Part #" "C105871"
 			(at 373.38 176.53 0)
 			(effects
@@
 			)
 		)
-		(property "Part" "0402WGF4701TCE"
+		(property "Part" "RC0402FR-074K7L"
 			(at 373.38 176.53 0)
 			(effects
@@
 			)
 		)
-		(property "JLCPCB Part #" "C25900"
+		(property "JLCPCB Part #" "C105871"
 			(at 373.38 165.1 0)
 			(effects
@@
 			)
 		)
-		(property "Part" "0402WGF4701TCE"
+		(property "Part" "RC0402FR-074K7L"
 			(at 373.38 165.1 0)
 			(effects
