File: eth_mcu.kicad_sch (KiCad schematic)
At the start: 44 parts, among them J10 RJ45_Hanrun_HR911105A_Horizon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, U55 LAN8742A, Y6 25Mhz

Commit message: bom: substitute out-of-stock semiconductors, fix Y6 case size
Semiconductor sweep (U/IC/Q/D/CR/SW, fan excluded). Stock verified against
live LCSC -- the JLCPCB parts-library snapshot proved unreliable in both
directions, e.g. BAS21 listed as 6 when it actually had 204,880, and the
Zynq listed as 84 when it had 2.

  U40  C411812  -> C164120   PM25LQ010B-SCE (1 in stock) -> W25X10CLSNIG-TR.
                             True drop-in: same 1Mbit density, SOIC-8 150mil,
                             2.3-3.6V, 104MHz, 25-series command set.

  U23  C393875  -> C2959323  S25FL128SAGMFI000 -> S25FL128SAGMFIR00.
                             Model R = SO-16 with RESET# and VIO, which is how
                             pin 3 (FLASH_RST_B) and pin 14 are already wired.
                             On the previous model-0 part both were RFU, so the
                             flash reset had never been functional. Sector type
                             unchanged (0 = uniform 64-KB hybrid), so the U-Boot
                             / MTD layout is unaffected, and Xilinx UG908 Table 44
                             lists s25fl128sxxxxxx0 as supported.

  Y6   C2901601 -> C17326988 SX2M25.000M20F30TNN -> SIT8008BI-21-YYS-25.000000.
                             The old part is a 2520 (2.5x2.0mm) oscillator on an
                             Abracon ASE 3.2x2.5mm land pattern; the new one is a
                             genuine 3225 part, so the existing footprint becomes
                             dimensionally correct. 25MHz +/-20ppm into the
                             LAN8742A reference, well inside the +/-50ppm that
                             100BASE-TX requires. No PCB change.

All three keep their existing footprints, so no re-routing is implied.

Also carries the netlist re-export and PCB sync for the earlier passives work,
which brought schematic, netlist and PCB into agreement across all 826 R/C.

NOTE: NASR.net and NASR.kicad_pcb predate the three substitutions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
Parts:
- Y6: JLCPCB Part # C2901601 -> C17326988; Part SX2M25.000M20F30TNN -> SIT8008BI-21-YYS-25.000000
Changed lines of the file:
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@@
 			)
 		)
-		(property "Description" "3.3V CMOS SMD Crystal Clock Oscillator"
+		(property "Description" "25MHz ±20ppm 1.62V~3.63V LVCMOS MEMS Oscillator SMD3225-4P ROHS"
 			(at 114.3 214.63 0)
 			(effects
@@
 			)
 		)
-		(property "Part" "SX2M25.000M20F30TNN"
+		(property "Part" "SIT8008BI-21-YYS-25.000000"
 			(at 114.3 214.63 0)
 			(effects
@@
 			)
 		)
-		(property "JLCPCB Part #" "C2901601"
+		(property "JLCPCB Part #" "C17326988"
 			(at 114.3 214.63 0)
 			(effects
