File: eth_mcu.kicad_sch (KiCad schematic)
At the start: 44 parts, among them J10 RJ45_Hanrun_HR911105A_Horizon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, U55 LAN8742A, Y6 25Mhz

Commit message: JLCPCB ID attribute updates
These 'JLCPCB Part #' updates reflect the JLCPCB assembly order # SMT026073061946-2250854A
Parts:
- R329: JLCPCB Part # C25852 -> C132157; Part 0402WGF1212TCE -> RC0402FR-0712K1L
Changed lines of the file:
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@@
 			)
 		)
-		(property "JLCPCB Part #" "C25852"
+		(property "JLCPCB Part #" "C132157"
 			(at 226.06 156.21 0)
 			(effects
@@
 			)
 		)
-		(property "Part" "0402WGF1212TCE"
+		(property "Part" "RC0402FR-0712K1L"
 			(at 226.06 156.21 0)
 			(effects
